Commit message: updated names for full robot

File: r2_description/urdf/r2_legs/r2_legs.left_foot.xacro (robot description, xacro)
@@ -51,5 +51,5 @@
     <limit effort="330.0" lower="-.5" upper=".5" velocity="1.0"/>
   </joint>
-  <joint name="${robot_name}left_leg/gripper/joint1" type="revolute">
+  <joint name="${robot_name}left_leg/gripper/jawLeft" type="revolute">
     <parent link="${robot_name}left_leg_foot"/>
     <child link="${robot_name}left_leg_jaw0"/>
@@ -59,5 +59,5 @@
     <limit effort="330.0" lower="-.5" upper=".5" velocity="1.0"/>
   </joint>
-  <joint name="${robot_name}left_leg/gripper/joint2" type="revolute">
+  <joint name="${robot_name}left_leg/gripper/jawRight" type="revolute">
     <parent link="${robot_name}left_leg_foot"/>
     <child link="${robot_name}left_leg_jaw1"/>

File: r2_description/urdf/r2_legs/r2_legs.right_foot.xacro (robot description, xacro)
@@ -52,5 +52,5 @@
     <limit effort="330.0" lower="-.5" upper=".5" velocity="1.0"/>
   </joint>
-  <joint name="${robot_name}right_leg/gripper/joint1" type="revolute">
+  <joint name="${robot_name}right_leg/gripper/jawLeft" type="revolute">
     <parent link="${robot_name}right_leg_foot"/>
     <child link="${robot_name}right_leg_jaw0"/>
@@ -61,5 +61,5 @@
     <traits spring_k="2.5"   />
   </joint>
-  <joint name="${robot_name}right_leg/gripper/joint2" type="revolute">
+  <joint name="${robot_name}right_leg/gripper/jawRight" type="revolute">
     <parent link="${robot_name}right_leg_foot"/>
     <child link="${robot_name}right_leg_jaw1"/>
