Commit message: reversed y axis on grippers so actual robot states matches

File: r2_description/urdf/r2c_legs/r2_legs.left_foot.xacro (robot description, xacro)
@@ -55,5 +55,5 @@
     <child link="${robot_name}left_leg_jaw0"/>
     <origin rpy="0.0 0 0" xyz="0.01905 0 0.17546"/>
-    <axis xyz="0 -1 0"/>
+    <axis xyz="0 1 0"/>
     <dynamics damping="${left_leg_gripper_j0_damping}" friction="${left_leg_gripper_j0_friction}"/>
     <limit effort="330.0" lower="-.5" upper=".5" velocity="1.0"/>
@@ -63,5 +63,5 @@
     <child link="${robot_name}left_leg_jaw1"/>
     <origin rpy="0.0 0 0" xyz="-0.01905 0 0.17546"/>
-    <axis xyz="0 1 0"/>
+    <axis xyz="0 -1 0"/>
     <dynamics damping="${left_leg_gripper_j1_damping}" friction="${left_leg_gripper_j1_friction}"/>
     <limit effort="330.0" lower="-.5" upper=".5" velocity="1.0"/>

File: r2_description/urdf/r2c_legs/r2_legs.right_foot.xacro (robot description, xacro)
@@ -56,5 +56,5 @@
     <child link="${robot_name}right_leg_jaw0"/>
     <origin rpy="0.0 0 0" xyz="0.01905 0 0.17546"/>
-    <axis xyz="0 -1 0"/>
+    <axis xyz="0 1 0"/>
     <dynamics damping="${right_leg_gripper_j0_damping}" friction="${right_leg_gripper_j0_friction}"/>
     <limit effort="330.0" lower="-.5" upper=".5" velocity="1.0"/>
@@ -65,5 +65,5 @@
     <child link="${robot_name}right_leg_jaw1"/>
     <origin rpy="0.0 0 0" xyz="-0.01905 0 0.17546"/>
-    <axis xyz="0 1 0"/>
+    <axis xyz="0 -1 0"/>
     <dynamics damping="${right_leg_gripper_j1_damping}" friction="${right_leg_gripper_j1_friction}"/>
     <limit effort="330.0" lower="-.5" upper=".5" velocity="1.0"/>
