Commit message: removed commented out portion of r2c.<hand>.xacro

File: r2_description/robots/xacro/r2_upperbody/r2c.left_hand.xacro (robot description, xacro)
@@ -15,8 +15,4 @@
   <property name="left_arm_hand_index_j2_damping" value= "0.1" />
   <property name="left_arm_hand_index_j2_friction" value= "0.0" />
-<!--
-  <property name="left_arm_hand_index_j3_damping" value= "0.1" />
-  <property name="left_arm_hand_index_j3_friction" value= "0.0" />
--->
   <property name="left_arm_hand_middle_j0_damping" value= "0.1" />
   <property name="left_arm_hand_middle_j0_friction" value= "0.0" />
@@ -25,24 +21,8 @@
   <property name="left_arm_hand_middle_j2_damping" value= "0.1" />
   <property name="left_arm_hand_middle_j2_friction" value= "0.0" />
-<!--
-  <property name="left_arm_hand_middle_j3_damping" value= "0.1" />
-  <property name="left_arm_hand_middle_j3_friction" value= "0.0" />
--->
   <property name="left_arm_hand_ring_j0_damping" value= "0.1" />
   <property name="left_arm_hand_ring_j0_friction" value= "0.0" />
-<!--
-  <property name="left_arm_hand_ring_j1_damping" value= "0.1" />
-  <property name="left_arm_hand_ring_j1_friction" value= "0.0" />
-  <property name="left_arm_hand_ring_j2_damping" value= "0.1" />
-  <property name="left_arm_hand_ring_j2_friction" value= "0.0" />
--->
   <property name="left_arm_hand_little_j0_damping" value= "0.1" />
   <property name="left_arm_hand_little_j0_friction" value= "0.0" />
-<!--
-  <property name="left_arm_hand_little_j1_damping" value= "0.1" />
-  <property name="left_arm_hand_little_j1_friction" value= "0.0" />
-  <property name="left_arm_hand_little_j2_damping" value= "0.1" />
-  <property name="left_arm_hand_little_j2_friction" value= "0.0" />
--->
   <joint name="${robot_name}left_arm/hand/thumb/roll" type="revolute">
     <parent link="${robot_name}left_wrist_yaw"/>
@@ -277,43 +257,4 @@
     </collision>
   </link>
-<!--
-  <joint name="${robot_name}left_arm/hand/index/distal" type="revolute">
-    <parent link="${robot_name}left_index_medial"/>
-    <child link="${robot_name}left_index_distal"/>
-    <origin xyz=" 0.03048 0.0 0.0 " rpy=" 0.0 0.0 0.0 " />
-    <axis xyz="0 0 1"/>
-    <limit effort="10000000.0" lower="0.0" upper="1.5708" velocity="1000"/>
-    <dynamics damping="${left_arm_hand_index_j3_damping}" friction="${left_arm_hand_index_j3_friction}"/>
-  </joint>
-  <link name="${robot_name}left_index_distal">
-    <inertial>
-      <mass value=".0010"/>
-      <inertia ixx=".0010" ixy="0.0" ixz="0.0" iyy=".0010" iyz="0.0" izz=".0010"/>
-    </inertial>
-    <visual>
-      <geometry>
-        <mesh filename="package://${resource_package}/meshes/r2_upperbody/Finger_Dist.dae"/>
-      </geometry>
-      <origin xyz="0.0 0.0 0.0" rpy="0 -1.57 0"/>
-    </visual>
-    <collision>
-      <geometry>
-        <mesh filename="package://${resource_package}/meshes/r2_upperbody/Finger_Dist.dae"/>
-      </geometry>
-      <origin xyz="0.0 0.0 0.0" rpy="0 -1.57 0"/>
-    </collision>
-  </link>
-  <joint name="${robot_name}fixed/left_index_distal/left_index_tip" type="fixed">
-    <parent link="${robot_name}left_index_distal"/>
-    <child link="${robot_name}left_index_tip"/>
-    <origin xyz=" 0.024638 0.0 0.0 " rpy=" 0.0 -0.0 0.0 " />
-  </joint>
-  <link name="${robot_name}left_index_tip">
-    <inertial>
-      <mass value=".0010"/>
-      <inertia ixx=".0010" ixy="0.0" ixz="0.0" iyy=".0010" iyz="0.0" izz=".0010"/>
-    </inertial>
-  </link>
--->
   <link name="${robot_name}left_middle_base">
     <inertial>
@@ -380,43 +321,4 @@
     </collision>
   </link>
-<!--
-  <joint name="${robot_name}left_arm/hand/middle/distal" type="revolute">
-    <parent link="${robot_name}left_middle_medial"/>
-    <child link="${robot_name}left_middle_distal"/>
-    <origin xyz=" 0.03048 0.0 0.0 " rpy=" 0.0 -0.0 0.0 " />
-    <axis xyz="0 0 1"/>
-    <limit effort="10000000.0" lower="0.0" upper="1.57" velocity="1000"/>
-    <dynamics damping="${left_arm_hand_middle_j3_damping}" friction="${left_arm_hand_middle_j3_friction}"/>
-  </joint>
-  <link name="${robot_name}left_middle_distal">
-    <inertial>
-      <mass value=".0010"/>
-      <inertia ixx=".0010" ixy="0.0" ixz="0.0" iyy=".0010" iyz="0.0" izz=".0010"/>
-    </inertial>
-    <visual>
-      <geometry>
-        <mesh filename="package://${resource_package}/meshes/r2_upperbody/Finger_Dist.dae"/>
-      </geometry>
-      <origin xyz="0.0 0.0 0.0" rpy="0 -1.57 0"/>
-    </visual>
-    <collision>
-      <geometry>
-        <mesh filename="package://${resource_package}/meshes/r2_upperbody/Finger_Dist.dae"/>
-      </geometry>
-      <origin xyz="0.0 0.0 0.0" rpy="0 -1.57 0"/>
-    </collision>
-  </link>
-  <joint name="${robot_name}fixed/left_middle_distal/left_middle_tip" type="fixed">
-    <parent link="${robot_name}left_middle_distal"/>
-    <child link="${robot_name}left_middle_tip"/>
-    <origin xyz=" 0.024638 0.0 0.0 " rpy=" 0.0 -0.0 0.0 " />
-  </joint>
-  <link name="${robot_name}left_middle_tip">
-    <inertial>
-      <mass value=".0010"/>
-      <inertia ixx=".0010" ixy="0.0" ixz="0.0" iyy=".0010" iyz="0.0" izz=".0010"/>
-    </inertial>
-  </link>
--->
   <link name="${robot_name}left_ring_proximal">
     <inertial>
@@ -437,69 +339,4 @@
     </collision>
   </link>
-<!--
-  <joint name="${robot_name}left_arm/hand/ringlittle/ringMedial" type="revolute">
-    <parent link="${robot_name}left_ring_proximal"/>
-    <child link="${robot_name}left_ring_medial"/>
-    <origin xyz=" 0.04445 0.0 0.0 " rpy=" 0.0 -0.0 0.0 " />
-    <axis xyz="0 0 1"/>
-    <limit effort="10000000.0" lower="0" upper="2.9671" velocity="1000"/>
-    <dynamics damping="${left_arm_hand_ring_j1_damping}" friction="${left_arm_hand_ring_j1_friction}"/>
-  </joint>
-  <link name="${robot_name}left_ring_medial">
-    <inertial>
-      <mass value=".0010"/>
-      <inertia ixx=".0010" ixy="0.0" ixz="0.0" iyy=".0010" iyz="0.0" izz=".0010"/>
-    </inertial>
-    <visual>
-      <geometry>
-        <mesh filename="package://${resource_package}/meshes/r2_upperbody/Finger_Mid.dae"/>
-      </geometry>
-      <origin xyz="0.0 0.0 0.0" rpy="3.14 0 1.57"/>
-    </visual>
-    <collision>
-      <geometry>
-        <mesh filename="package://${resource_package}/meshes/r2_upperbody/Finger_Mid.dae"/>
-      </geometry>
-      <origin xyz="0.0 0.0 0.0" rpy="3.14 0 1.57"/>
-    </collision>
-  </link>
-  <joint name="${robot_name}left_arm/hand/ringlittle/ringDistal" type="revolute">
-    <parent link="${robot_name}left_ring_medial"/>
-    <child link="${robot_name}left_ring_distal"/>
-    <origin xyz=" 0.03048 0.0 0.0 " rpy=" 0.0 -0.0 0.0 " />
-    <axis xyz="0 0 1"/>
-    <limit effort="10000000.0" lower="0" upper="2.9671" velocity="1000"/>
-    <dynamics damping="${left_arm_hand_ring_j2_damping}" friction="${left_arm_hand_ring_j2_friction}"/>
-  </joint>
-  <link name="${robot_name}left_ring_distal">
-    <inertial>
-      <mass value=".0010"/>
-      <inertia ixx=".0010" ixy="0.0" ixz="0.0" iyy=".0010" iyz="0.0" izz=".0010"/>
-    </inertial>
-    <visual>
-      <geometry>
-        <mesh filename="package://${resource_package}/meshes/r2_upperbody/Finger_Dist.dae"/>
-      </geometry>
-      <origin xyz="0.0 0.0 0.0" rpy="0 -1.57 0"/>
-    </visual>
-    <collision>
-      <geometry>
-        <mesh filename="package://${resource_package}/meshes/r2_upperbody/Finger_Dist.dae"/>
-      </geometry>
-      <origin xyz="0.0 0.0 0.0" rpy="0 -1.57 0"/>
-    </collision>
-  </link>
-  <joint name="${robot_name}fixed/left_ring_distal/left_ring_tip" type="fixed">
-    <parent link="${robot_name}left_ring_distal"/>
-    <child link="${robot_name}left_ring_tip"/>
-    <origin xyz=" 0.024638 0.0 0.0 " rpy=" 0.0 -0.0 0.0 " />
-  </joint>
-  <link name="${robot_name}left_ring_tip">
-    <inertial>
-      <mass value=".0010"/>
-      <inertia ixx=".0010" ixy="0.0" ixz="0.0" iyy=".0010" iyz="0.0" izz=".0010"/>
-    </inertial>
-  </link>
--->
   <link name="${robot_name}left_little_proximal">
     <inertial>
@@ -520,68 +357,3 @@
     </collision>
   </link>
-<!--
-  <joint name="${robot_name}left_arm/hand/ringlittle/littleMedial" type="revolute">
-    <parent link="${robot_name}left_little_proximal"/>
-    <child link="${robot_name}left_little_medial"/>
-    <origin xyz=" 0.04445 0.0 0.0 " rpy=" 0.0 -0.0 0.0 " />
-    <axis xyz="0 0 1"/>
-    <limit effort="10000000.0" lower="0" upper="2.9671" velocity="1000"/>
-    <dynamics damping="${left_arm_hand_little_j1_damping}" friction="${left_arm_hand_little_j1_friction}"/>
-  </joint>
-  <link name="${robot_name}left_little_medial">
-    <inertial>
-      <mass value=".0010"/>
-      <inertia ixx=".0010" ixy="0.0" ixz="0.0" iyy=".0010" iyz="0.0" izz=".0010"/>
-    </inertial>
-    <visual>
-      <geometry>
-        <mesh filename="package://${resource_package}/meshes/r2_upperbody/Finger_Mid.dae"/>
-      </geometry>
-      <origin xyz="0.0 0.0 0.0" rpy="3.14 0 1.57"/>
-    </visual>
-    <collision>
-      <geometry>
-        <mesh filename="package://${resource_package}/meshes/r2_upperbody/Finger_Mid.dae"/>
-      </geometry>
-      <origin xyz="0.0 0.0 0.0" rpy="3.14 0 1.57"/>
-    </collision>
-  </link>
-  <joint name="${robot_name}left_arm/hand/ringlittle/littleDistal" type="revolute">
-    <parent link="${robot_name}left_little_medial"/>
-    <child link="${robot_name}left_little_distal"/>
-    <origin xyz=" 0.03048 0.0 0.0 " rpy=" 0.0 -0.0 0.0 " />
-    <axis xyz="0 0 1"/>
-    <limit effort="10000000.0" lower="0" upper="2.9671" velocity="1000"/>
-    <dynamics damping="${left_arm_hand_little_j2_damping}" friction="${left_arm_hand_little_j2_friction}"/>
-  </joint>
-  <link name="${robot_name}left_little_distal">
-    <inertial>
-      <mass value=".0010"/>
-      <inertia ixx=".0010" ixy="0.0" ixz="0.0" iyy=".0010" iyz="0.0" izz=".0010"/>
-    </inertial>
-    <visual>
-      <geometry>
-        <mesh filename="package://${resource_package}/meshes/r2_upperbody/Finger_Dist.dae"/>
-      </geometry>
-      <origin xyz="0.0 0.0 0.0" rpy="0 -1.57 0"/>
-    </visual>
-    <collision>
-      <geometry>
-        <mesh filename="package://${resource_package}/meshes/r2_upperbody/Finger_Dist.dae"/>
-      </geometry>
-      <origin xyz="0.0 0.0 0.0" rpy="0 -1.57 0"/>
-    </collision>
-  </link>
-  <joint name="${robot_name}fixed/left_little_distal/left_little_tip" type="fixed">
-    <parent link="${robot_name}left_little_distal"/>
-    <child link="${robot_name}left_little_tip"/>
-    <origin xyz=" 0.024638 0.0 0.0 " rpy=" 0.0 -0.0 0.0 " />
-  </joint>
-  <link name="${robot_name}left_little_tip">
-    <inertial>
-      <mass value=".0010"/>
-      <inertia ixx=".0010" ixy="0.0" ixz="0.0" iyy=".0010" iyz="0.0" izz=".0010"/>
-    </inertial>
-  </link>
--->
 </robot>

File: r2_description/robots/xacro/r2_upperbody/r2c.right_hand.xacro (robot description, xacro)
@@ -15,8 +15,4 @@
   <property name="right_arm_hand_index_j2_damping" value= "0.1" />
   <property name="right_arm_hand_index_j2_friction" value= "0.0" />
-<!--
-  <property name="right_arm_hand_index_j3_damping" value= "0.1" />
-  <property name="right_arm_hand_index_j3_friction" value= "0.0" />
--->
   <property name="right_arm_hand_middle_j0_damping" value= "0.1" />
   <property name="right_arm_hand_middle_j0_friction" value= "0.0" />
@@ -25,24 +21,8 @@
   <property name="right_arm_hand_middle_j2_damping" value= "0.1" />
   <property name="right_arm_hand_middle_j2_friction" value= "0.0" />
-<!--
-  <property name="right_arm_hand_middle_j3_damping" value= "0.1" />
-  <property name="right_arm_hand_middle_j3_friction" value= "0.0" />
--->
   <property name="right_arm_hand_ring_j0_damping" value= "0.1" />
   <property name="right_arm_hand_ring_j0_friction" value= "0.0" />
-<!--
-  <property name="right_arm_hand_ring_j1_damping" value= "0.1" />
-  <property name="right_arm_hand_ring_j1_friction" value= "0.0" />
-  <property name="right_arm_hand_ring_j2_damping" value= "0.1" />
-  <property name="right_arm_hand_ring_j2_friction" value= "0.0" />
--->
   <property name="right_arm_hand_little_j0_damping" value= "0.1" />
   <property name="right_arm_hand_little_j0_friction" value= "0.0" />
-<!--
-  <property name="right_arm_hand_little_j1_damping" value= "0.1" />
-  <property name="right_arm_hand_little_j1_friction" value= "0.0" />
-  <property name="right_arm_hand_little_j2_damping" value= "0.1" />
-  <property name="right_arm_hand_little_j2_friction" value= "0.0" />
--->
 <joint name="${robot_name}right_arm/hand/thumb/roll" type="revolute">
     <parent link="${robot_name}right_wrist_yaw"/>
@@ -277,43 +257,4 @@
     </collision>
   </link>
-<!--
-  <joint name="${robot_name}right_arm/hand/index/distal" type="revolute">
-    <parent link="${robot_name}right_index_medial"/>
-    <child link="${robot_name}right_index_distal"/>
-    <origin xyz=" 0.03048 0.0 0.0 " rpy=" 0.0 0.0 0.0 " />
-    <axis xyz="0 0 1"/>
-    <limit effort="10000000.0" lower="0.0" upper="1.5708" velocity="1000"/>
-    <dynamics damping="${right_arm_hand_index_j3_damping}" friction="${right_arm_hand_index_j3_friction}"/>
-  </joint>
-  <link name="${robot_name}right_index_distal">
-    <inertial>
-      <mass value=".05"/>
-      <inertia ixx=".0010" ixy="0.0" ixz="0.0" iyy=".0010" iyz="0.0" izz=".0010"/>
-    </inertial>
-    <visual>
-      <geometry>
-        <mesh filename="package://${resource_package}/meshes/r2_upperbody/Finger_Dist.dae"/>
-      </geometry>
-      <origin xyz="0.0 0.0 0.0" rpy="0 -1.57 0"/>
-    </visual>
-    <collision>
-      <geometry>
-        <mesh filename="package://${resource_package}/meshes/r2_upperbody/Finger_Dist.dae"/>
-      </geometry>
-      <origin xyz="0.0 0.0 0.0" rpy="0 -1.57 0"/>
-    </collision>
-  </link>
-  <joint name="${robot_name}fixed/right_index_distal/right_index_tip" type="fixed">
-    <parent link="${robot_name}right_index_distal"/>
-    <child link="${robot_name}right_index_tip"/>
-    <origin xyz=" 0.024638 0.0 0.0 " rpy=" 0.0 -0.0 0.0 " />
-  </joint>
-  <link name="${robot_name}right_index_tip">
-    <inertial>
-      <mass value=".05"/>
-      <inertia ixx=".0010" ixy="0.0" ixz="0.0" iyy=".0010" iyz="0.0" izz=".0010"/>
-    </inertial>
-  </link>
--->
   <link name="${robot_name}right_middle_base">
     <inertial>
@@ -380,43 +321,4 @@
     </collision>
   </link>
-<!--
-  <joint name="${robot_name}right_arm/hand/middle/distal" type="revolute">
-    <parent link="${robot_name}right_middle_medial"/>
-    <child link="${robot_name}right_middle_distal"/>
-    <origin xyz=" 0.03048 0.0 0.0 " rpy=" 0.0 0.0 0.0 " />
-    <axis xyz="0 0 1"/>
-    <limit effort="10000000.0" lower="0.0" upper="1.5708" velocity="1000"/>
-    <dynamics damping="${right_arm_hand_middle_j3_damping}" friction="${right_arm_hand_middle_j3_friction}"/>
-  </joint>
-  <link name="${robot_name}right_middle_distal">
-    <inertial>
-      <mass value=".05"/>
-      <inertia ixx=".0010" ixy="0.0" ixz="0.0" iyy=".0010" iyz="0.0" izz=".0010"/>
-    </inertial>
-    <visual>
-      <geometry>
-        <mesh filename="package://${resource_package}/meshes/r2_upperbody/Finger_Dist.dae"/>
-      </geometry>
-      <origin xyz="0.0 0.0 0.0" rpy="0 -1.57 0"/>
-    </visual>
-    <collision>
-      <geometry>
-        <mesh filename="package://${resource_package}/meshes/r2_upperbody/Finger_Dist.dae" scale="0.9 0.9 0.9"/>
-      </geometry>
-      <origin xyz="0.0 0.0 0.0" rpy="0 -1.57 0"/>
-    </collision>
-  </link>
-  <joint name="${robot_name}fixed/right_middle_distal/right_middle_tip" type="fixed">
-    <parent link="${robot_name}right_middle_distal"/>
-    <child link="${robot_name}right_middle_tip"/>
-    <origin xyz=" 0.024638 0.0 0.0 " rpy=" 0.0 -0.0 0.0 " />
-  </joint>
-  <link name="${robot_name}right_middle_tip">
-    <inertial>
-      <mass value=".05"/>
-      <inertia ixx=".0010" ixy="0.0" ixz="0.0" iyy=".0010" iyz="0.0" izz=".0010"/>
-    </inertial>
-  </link>
--->
   <link name="${robot_name}right_ring_proximal">
     <inertial>
@@ -437,69 +339,4 @@
     </collision>
   </link>
-<!--
-  <joint name="${robot_name}right_arm/hand/ringlittle/ringMedial" type="revolute">
-    <parent link="${robot_name}right_ring_proximal"/>
-    <child link="${robot_name}right_ring_medial"/>
-    <origin xyz=" 0.04445 0.0 0.0 " rpy=" 0.0 -0.0 0.0 " />
-    <axis xyz="0 0 1"/>
-    <limit effort="10000000.0" lower="0" upper="2.9671" velocity="1000"/>
-    <dynamics damping="${right_arm_hand_ring_j1_damping}" friction="${right_arm_hand_ring_j1_friction}"/>
-  </joint>
-  <link name="${robot_name}right_ring_medial">
-    <inertial>
-      <mass value=".05"/>
-      <inertia ixx=".0010" ixy="0.0" ixz="0.0" iyy=".0010" iyz="0.0" izz=".0010"/>
-    </inertial>
-    <visual>
-      <geometry>
-        <mesh filename="package://${resource_package}/meshes/r2_upperbody/Finger_Mid.dae"/>
-      </geometry>
-      <origin xyz="0.0 0.0 0.0" rpy="3.14 0 1.57"/>
-    </visual>
-    <collision>
-      <geometry>
-        <mesh filename="package://${resource_package}/meshes/r2_upperbody/Finger_Mid.dae" scale="0.9 0.9 0.9"/>
-      </geometry>
-      <origin xyz="0.0 0.0 0.0" rpy="3.14 0 1.57"/>
-    </collision>
-  </link>
-  <joint name="${robot_name}right_arm/hand/ringlittle/ringDistal" type="revolute">
-    <parent link="${robot_name}right_ring_medial"/>
-    <child link="${robot_name}right_ring_distal"/>
-    <origin xyz=" 0.03048 0.0 0.0 " rpy=" 0.0 -0.0 0.0 " />
-    <axis xyz="0 0 1"/>
-    <limit effort="10000000.0" lower="0" upper="2.9671" velocity="1000"/>
-    <dynamics damping="${right_arm_hand_ring_j2_damping}" friction="${right_arm_hand_ring_j2_friction}"/>
-  </joint>
-  <link name="${robot_name}right_ring_distal">
-    <inertial>
-      <mass value=".05"/>
-      <inertia ixx=".0010" ixy="0.0" ixz="0.0" iyy=".0010" iyz="0.0" izz=".0010"/>
-    </inertial>
-    <visual>
-      <geometry>
-        <mesh filename="package://${resource_package}/meshes/r2_upperbody/Finger_Dist.dae"/>
-      </geometry>
-      <origin xyz="0.0 0.0 0.0" rpy="0 -1.57 0"/>
-    </visual>
-    <collision>
-      <geometry>
-        <mesh filename="package://${resource_package}/meshes/r2_upperbody/Finger_Dist.dae" scale="0.9 0.9 0.9"/>
-      </geometry>
-      <origin xyz="0.0 0.0 0.0" rpy="0 -1.57 0"/>
-    </collision>
-  </link>
-  <joint name="${robot_name}fixed/right_ring_distal/right_ring_tip" type="fixed">
-    <parent link="${robot_name}right_ring_distal"/>
-    <child link="${robot_name}right_ring_tip"/>
-    <origin xyz=" 0.024638 0.0 0.0 " rpy=" 0.0 -0.0 0.0 " />
-  </joint>
-  <link name="${robot_name}right_ring_tip">
-    <inertial>
-      <mass value=".05"/>
-      <inertia ixx=".0010" ixy="0.0" ixz="0.0" iyy=".0010" iyz="0.0" izz=".0010"/>
-    </inertial>
-  </link>
--->
   <link name="${robot_name}right_little_proximal">
     <inertial>
@@ -520,68 +357,3 @@
     </collision>
   </link>
-<!--
-  <joint name="${robot_name}right_arm/hand/ringlittle/littleMedial" type="revolute">
-    <parent link="${robot_name}right_little_proximal"/>
-    <child link="${robot_name}right_little_medial"/>
-    <origin xyz=" 0.04445 0.0 0.0 " rpy=" 0.0 -0.0 0.0 " />
-    <axis xyz="0 0 1"/>
-    <limit effort="10000000.0" lower="0" upper="2.9671" velocity="1000"/>
-    <dynamics damping="${right_arm_hand_little_j1_damping}" friction="${right_arm_hand_little_j1_friction}"/>
-  </joint>
-  <link name="${robot_name}right_little_medial">
-    <inertial>
-      <mass value=".05"/>
-      <inertia ixx=".0010" ixy="0.0" ixz="0.0" iyy=".0010" iyz="0.0" izz=".0010"/>
-    </inertial>
-    <visual>
-      <geometry>
-        <mesh filename="package://${resource_package}/meshes/r2_upperbody/Finger_Mid.dae"/>
-      </geometry>
-      <origin xyz="0.0 0.0 0.0" rpy="3.14 0 1.57"/>
-    </visual>
-    <collision>
-      <geometry>
-        <mesh filename="package://${resource_package}/meshes/r2_upperbody/Finger_Mid.dae" scale="0.9 0.9 0.9"/>
-      </geometry>
-      <origin xyz="0.0 0.0 0.0" rpy="3.14 0 1.57"/>
-    </collision>
-  </link>
-  <joint name="${robot_name}right_arm/hand/ringlittle/littleDistal" type="revolute">
-    <parent link="${robot_name}right_little_medial"/>
-    <child link="${robot_name}right_little_distal"/>
-    <origin xyz=" 0.03048 0.0 0.0 " rpy=" 0.0 -0.0 0.0 " />
-    <axis xyz="0 0 1"/>
-    <limit effort="10000000.0" lower="0" upper="2.9671" velocity="1000"/>
-    <dynamics damping="${right_arm_hand_little_j2_damping}" friction="${right_arm_hand_little_j2_friction}"/>
-  </joint>
-  <link name="${robot_name}right_little_distal">
-    <inertial>
-      <mass value=".05"/>
-      <inertia ixx=".0010" ixy="0.0" ixz="0.0" iyy=".0010" iyz="0.0" izz=".0010"/>
-    </inertial>
-    <visual>
-      <geometry>
-        <mesh filename="package://${resource_package}/meshes/r2_upperbody/Finger_Dist.dae"/>
-      </geometry>
-      <origin xyz="0.0 0.0 0.0" rpy="0 -1.57 0"/>
-    </visual>
-    <collision>
-      <geometry>
-        <mesh filename="package://${resource_package}/meshes/r2_upperbody/Finger_Dist.dae" scale="0.9 0.9 0.9"/>
-      </geometry>
-      <origin xyz="0.0 0.0 0.0" rpy="0 -1.57 0"/>
-    </collision>
-  </link>
-  <joint name="${robot_name}fixed/right_little_distal/right_little_tip" type="fixed">
-    <parent link="${robot_name}right_little_distal"/>
-    <child link="${robot_name}right_little_tip"/>
-    <origin xyz=" 0.024638 0.0 0.0 " rpy=" 0.0 -0.0 0.0 " />
-  </joint>
-  <link name="${robot_name}right_little_tip">
-    <inertial>
-      <mass value=".05"/>
-      <inertia ixx=".0010" ixy="0.0" ixz="0.0" iyy=".0010" iyz="0.0" izz=".0010"/>
-    </inertial>
-  </link>
--->
 </robot>
