Commit message: updated urdf ringlittle joint

File: r2_description/urdf/r2.left_hand.xacro (robot description, xacro)
@@ -71,5 +71,5 @@
     <dynamics damping="${left_arm_hand_middle_j0_damping}" friction="${left_arm_hand_middle_j0_friction}"/>
   </joint>
-  <joint name="${robot_name}left_arm/hand/ring/proximal" type="revolute">
+  <joint name="${robot_name}left_arm/hand/ringlittle/ring" type="revolute">
     <parent link="${robot_name}left_wrist_yaw"/>
     <child link="${robot_name}left_ring_proximal"/>
@@ -79,5 +79,5 @@
     <dynamics damping="${left_arm_hand_ring_j0_damping}" friction="${left_arm_hand_ring_j0_friction}"/>
   </joint>
-  <joint name="${robot_name}left_arm/hand/little/proximal" type="revolute">
+  <joint name="${robot_name}left_arm/hand/ringlittle/little" type="revolute">
     <parent link="${robot_name}left_wrist_yaw"/>
     <child link="${robot_name}left_little_proximal"/>
@@ -425,5 +425,5 @@
     </collision>
   </link>
-  <joint name="${robot_name}left_arm/hand/ring/medial" type="revolute">
+  <joint name="${robot_name}left_arm/hand/ringlittle/ringMedial" type="revolute">
     <parent link="${robot_name}left_ring_proximal"/>
     <child link="${robot_name}left_ring_medial"/>
@@ -451,5 +451,5 @@
     </collision>
   </link>
-  <joint name="${robot_name}left_arm/hand/ring/distal" type="revolute">
+  <joint name="${robot_name}left_arm/hand/ringlittle/ringDistal" type="revolute">
     <parent link="${robot_name}left_ring_medial"/>
     <child link="${robot_name}left_ring_distal"/>
@@ -506,5 +506,5 @@
     </collision>
   </link>
-  <joint name="${robot_name}left_arm/hand/little/medial" type="revolute">
+  <joint name="${robot_name}left_arm/hand/ringlittle/littleMedial" type="revolute">
     <parent link="${robot_name}left_little_proximal"/>
     <child link="${robot_name}left_little_medial"/>
@@ -532,5 +532,5 @@
     </collision>
   </link>
-  <joint name="${robot_name}left_arm/hand/little/distal" type="revolute">
+  <joint name="${robot_name}left_arm/hand/ringlittle/littleDistal" type="revolute">
     <parent link="${robot_name}left_little_medial"/>
     <child link="${robot_name}left_little_distal"/>

File: r2_description/urdf/r2.right_hand.xacro (robot description, xacro)
@@ -71,5 +71,5 @@
     <dynamics damping="${right_arm_hand_middle_j0_damping}" friction="${right_arm_hand_middle_j0_friction}"/>
   </joint>
-  <joint name="${robot_name}right_arm/hand/ring/proximal" type="revolute">
+  <joint name="${robot_name}right_arm/hand/ringlittle/ring" type="revolute">
     <parent link="${robot_name}right_wrist_yaw"/>
     <child link="${robot_name}right_ring_proximal"/>
@@ -79,5 +79,5 @@
     <dynamics damping="${right_arm_hand_ring_j0_damping}" friction="${right_arm_hand_ring_j0_friction}"/>
   </joint>
-  <joint name="${robot_name}right_arm/hand/little/proximal" type="revolute">
+  <joint name="${robot_name}right_arm/hand/ringlittle/little" type="revolute">
     <parent link="${robot_name}right_wrist_yaw"/>
     <child link="${robot_name}right_little_proximal"/>
@@ -425,5 +425,5 @@
     </collision>
   </link>
-  <joint name="${robot_name}right_arm/hand/ring/medial" type="revolute">
+  <joint name="${robot_name}right_arm/hand/ringlittle/ringMedial" type="revolute">
     <parent link="${robot_name}right_ring_proximal"/>
     <child link="${robot_name}right_ring_medial"/>
@@ -451,5 +451,5 @@
     </collision>
   </link>
-  <joint name="${robot_name}right_arm/hand/ring/distal" type="revolute">
+  <joint name="${robot_name}right_arm/hand/ringlittle/ringDistal" type="revolute">
     <parent link="${robot_name}right_ring_medial"/>
     <child link="${robot_name}right_ring_distal"/>
@@ -506,5 +506,5 @@
     </collision>
   </link>
-  <joint name="${robot_name}right_arm/hand/little/medial" type="revolute">
+  <joint name="${robot_name}right_arm/hand/ringlittle/littleMedial" type="revolute">
     <parent link="${robot_name}right_little_proximal"/>
     <child link="${robot_name}right_little_medial"/>
@@ -532,5 +532,5 @@
     </collision>
   </link>
-  <joint name="${robot_name}right_arm/hand/little/distal" type="revolute">
+  <joint name="${robot_name}right_arm/hand/ringlittle/littleDistal" type="revolute">
     <parent link="${robot_name}right_little_medial"/>
     <child link="${robot_name}right_little_distal"/>
