Commit message: simplified finger meshes and added some more grasps to srdf

File: r2_description/urdf/r2.left_hand.xacro (robot description, xacro)
@@ -1,39 +1,39 @@
 <?xml version="1.0"?>
 <robot>
-  <property name="left_arm_hand_thumb_j0_damping" value= "0.1" />
+  <property name="left_arm_hand_thumb_j0_damping" value= "0.5" />
   <property name="left_arm_hand_thumb_j0_friction" value= "0.0" />
-  <property name="left_arm_hand_thumb_j1_damping" value= "0.1" />
+  <property name="left_arm_hand_thumb_j1_damping" value= "0.5" />
   <property name="left_arm_hand_thumb_j1_friction" value= "0.0" />
-  <property name="left_arm_hand_thumb_j2_damping" value= "0.1" />
+  <property name="left_arm_hand_thumb_j2_damping" value= "0.5" />
   <property name="left_arm_hand_thumb_j2_friction" value= "0.0" />
-  <property name="left_arm_hand_thumb_j3_damping" value= "0.1" />
+  <property name="left_arm_hand_thumb_j3_damping" value= "0.5" />
   <property name="left_arm_hand_thumb_j3_friction" value= "0.0" />
-  <property name="left_arm_hand_index_j0_damping" value= "0.1" />
+  <property name="left_arm_hand_index_j0_damping" value= "0.5" />
   <property name="left_arm_hand_index_j0_friction" value= "0.0" />
-  <property name="left_arm_hand_index_j1_damping" value= "0.1" />
+  <property name="left_arm_hand_index_j1_damping" value= "0.5" />
   <property name="left_arm_hand_index_j1_friction" value= "0.0" />
-  <property name="left_arm_hand_index_j2_damping" value= "0.1" />
+  <property name="left_arm_hand_index_j2_damping" value= "0.5" />
   <property name="left_arm_hand_index_j2_friction" value= "0.0" />
-  <property name="left_arm_hand_index_j3_damping" value= "0.1" />
+  <property name="left_arm_hand_index_j3_damping" value= "0.5" />
   <property name="left_arm_hand_index_j3_friction" value= "0.0" />
-  <property name="left_arm_hand_middle_j0_damping" value= "0.1" />
+  <property name="left_arm_hand_middle_j0_damping" value= "0.5" />
   <property name="left_arm_hand_middle_j0_friction" value= "0.0" />
-  <property name="left_arm_hand_middle_j1_damping" value= "0.1" />
+  <property name="left_arm_hand_middle_j1_damping" value= "0.5" />
   <property name="left_arm_hand_middle_j1_friction" value= "0.0" />
-  <property name="left_arm_hand_middle_j2_damping" value= "0.1" />
+  <property name="left_arm_hand_middle_j2_damping" value= "0.5" />
   <property name="left_arm_hand_middle_j2_friction" value= "0.0" />
-  <property name="left_arm_hand_middle_j3_damping" value= "0.1" />
+  <property name="left_arm_hand_middle_j3_damping" value= "0.5" />
   <property name="left_arm_hand_middle_j3_friction" value= "0.0" />
-  <property name="left_arm_hand_ring_j0_damping" value= "0.1" />
+  <property name="left_arm_hand_ring_j0_damping" value= "0.5" />
   <property name="left_arm_hand_ring_j0_friction" value= "0.0" />
-  <property name="left_arm_hand_ring_j1_damping" value= "0.1" />
+  <property name="left_arm_hand_ring_j1_damping" value= "0.5" />
   <property name="left_arm_hand_ring_j1_friction" value= "0.0" />
-  <property name="left_arm_hand_ring_j2_damping" value= "0.1" />
+  <property name="left_arm_hand_ring_j2_damping" value= "0.5" />
   <property name="left_arm_hand_ring_j2_friction" value= "0.0" />
-  <property name="left_arm_hand_little_j0_damping" value= "0.1" />
+  <property name="left_arm_hand_little_j0_damping" value= "0.5" />
   <property name="left_arm_hand_little_j0_friction" value= "0.0" />
-  <property name="left_arm_hand_little_j1_damping" value= "0.1" />
+  <property name="left_arm_hand_little_j1_damping" value= "0.5" />
   <property name="left_arm_hand_little_j1_friction" value= "0.0" />
-  <property name="left_arm_hand_little_j2_damping" value= "0.1" />
+  <property name="left_arm_hand_little_j2_damping" value= "0.5" />
   <property name="left_arm_hand_little_j2_friction" value= "0.0" />
   <joint name="${robot_name}left_arm/hand/thumb/joint0" type="revolute">
@@ -109,10 +109,10 @@
       <origin xyz="-0.01 0.0 0.0" rpy="-1.57 0 0"/>
     </visual>
-    <collision>
+   <!--  <collision>
       <geometry>
         <mesh filename="package://r2_description/meshes/Left_Thumb_Carp.dae"/>
       </geometry>
       <origin xyz="-0.01 0.0 0.0" rpy="-1.57 0 0"/>
-    </collision>
+    </collision> -->
   </link>
   <joint name="${robot_name}left_arm/hand/thumb/joint1" type="revolute">
@@ -137,7 +137,9 @@
     <collision>
       <geometry>
-        <mesh filename="package://r2_description/meshes/Left_Thumb_MtCar.dae"/>
-      </geometry>
-      <origin xyz="0.0 0.0 0.0" rpy="-1.57 -1.57 0"/>
+ <!--        <mesh filename="package://r2_description/meshes/Left_Thumb_MtCar.dae"/> -->
+        <box size="0.01 0.02 0.01" />
+      </geometry>
+<!--       <origin xyz="0.0 0.0 0.0" rpy="-1.57 -1.57 0"/> -->
+      <origin xyz="0.02 0.0 0.0" rpy="-1.57 -1.57 0"/>
     </collision>
   </link>
@@ -163,7 +165,9 @@
     <collision>
       <geometry>
-        <mesh filename="package://r2_description/meshes/Thumb_Proximal.dae"/>
-      </geometry>
-      <origin xyz="0.0 0.0 0.0" rpy="3.14 0 1.57"/>
+<!--         <mesh filename="package://r2_description/meshes/Thumb_Proximal.dae"/> -->
+          <box size="0.01 0.03 0.01" />
+      </geometry>
+<!--       <origin xyz="0.0 0.0 0.0" rpy="3.14 0 1.57"/> -->
+      <origin xyz="0.022 0.0 0.0" rpy="3.14 0 1.57"/>
     </collision>
   </link>
@@ -189,7 +193,9 @@
     <collision>
       <geometry>
-        <mesh filename="package://r2_description/meshes/Thumb_Dist.dae"/>
-      </geometry>
-      <origin xyz="0.0 0.0 0.0" rpy="3.14 3.14 0"/>
+<!--         <mesh filename="package://r2_description/meshes/Thumb_Dist.dae"/> -->
+        <box size="0.025 0.01 0.01" />
+      </geometry>
+ <!--      <origin xyz="0.0 0.0 0.0" rpy="3.14 3.14 0"/> -->
+      <origin xyz="0.015 0.0 0.0" rpy="3.14 3.14 0"/>
     </collision>
   </link>
@@ -238,7 +244,9 @@
     <collision>
       <geometry>
-        <mesh filename="package://r2_description/meshes/Finger_Proximal.dae"/>
-      </geometry>
-      <origin xyz="0.0 0.0 0.0" rpy="0 0 1.57"/>
+<!--         <mesh filename="package://r2_description/meshes/Finger_Proximal.dae"/> -->
+         <box size="0.01 0.04 0.01" />
+      </geometry>
+      <origin xyz="0.02 0.0 0.0" rpy="0 0 1.57"/>
+<!--       <origin xyz="0.0 0.0 0.0" rpy="0 0 1.57"/> -->
     </collision>
   </link>
@@ -264,7 +272,9 @@
     <collision>
       <geometry>
-        <mesh filename="package://r2_description/meshes/Finger_Mid.dae"/>
-      </geometry>
-      <origin xyz="0.0 0.0 0.0" rpy="3.14 0 1.57"/>
+<!--         <mesh filename="package://r2_description/meshes/Finger_Mid.dae"/> -->
+        <box size="0.01 0.025 0.01" />
+      </geometry>
+<!--       <origin xyz="0.0 0.0 0.0" rpy="3.14 0 1.57"/> -->
+      <origin xyz="0.0125 0.0 0.0" rpy="3.14 0 1.57"/>
     </collision>
   </link>
@@ -290,7 +300,9 @@
     <collision>
       <geometry>
-        <mesh filename="package://r2_description/meshes/Finger_Dist.dae"/>
-      </geometry>
-      <origin xyz="0.0 0.0 0.0" rpy="0 -1.57 0"/>
+<!--         <mesh filename="package://r2_description/meshes/Finger_Dist.dae"/> -->
+        <box size="0.01 0.01 0.02" />
+      </geometry>
+<!--       <origin xyz="0.0 0.0 0.0" rpy="0 -1.57 0"/> -->
+      <origin xyz="0.015 0.0 0.0" rpy="0 -1.57 0"/>
     </collision>
   </link>
@@ -339,7 +351,9 @@
     <collision>
       <geometry>
-        <mesh filename="package://r2_description/meshes/Finger_Proximal.dae"/>
-      </geometry>
-      <origin xyz="0.0 0.0 0.0" rpy="0 0 1.57"/>
+     <!--    <mesh filename="package://r2_description/meshes/Finger_Proximal.dae"/> -->
+       <box size="0.01 0.04 0.01" />
+      </geometry>
+<!--       <origin xyz="0.0 0.0 0.0" rpy="0 0 1.57"/> -->
+      <origin xyz="0.02 0.0 0.0" rpy="0 0 1.57"/>
     </collision>
   </link>
@@ -363,9 +377,11 @@
       <origin xyz="0.0 0.0 0.0" rpy="3.14 0 1.57"/>
     </visual>
-    <collision>
-      <geometry>
-        <mesh filename="package://r2_description/meshes/Finger_Mid.dae"/>
-      </geometry>
-      <origin xyz="0.0 0.0 0.0" rpy="3.14 0 1.57"/>
+   <collision>
+      <geometry>
+<!--         <mesh filename="package://r2_description/meshes/Finger_Mid.dae"/> -->
+        <box size="0.01 0.025 0.01" />
+      </geometry>
+<!--       <origin xyz="0.0 0.0 0.0" rpy="3.14 0 1.57"/> -->
+      <origin xyz="0.0125 0.0 0.0" rpy="3.14 0 1.57"/>
     </collision>
   </link>
@@ -389,9 +405,11 @@
       <origin xyz="0.0 0.0 0.0" rpy="0 -1.57 0"/>
     </visual>
-    <collision>
-      <geometry>
-        <mesh filename="package://r2_description/meshes/Finger_Dist.dae"/>
-      </geometry>
-      <origin xyz="0.0 0.0 0.0" rpy="0 -1.57 0"/>
+   <collision>
+      <geometry>
+<!--         <mesh filename="package://r2_description/meshes/Finger_Dist.dae"/> -->
+        <box size="0.01 0.01 0.02" />
+      </geometry>
+<!--       <origin xyz="0.0 0.0 0.0" rpy="0 -1.57 0"/> -->
+      <origin xyz="0.015 0.0 0.0" rpy="0 -1.57 0"/>
     </collision>
   </link>
@@ -420,7 +438,9 @@
     <collision>
       <geometry>
-        <mesh filename="package://r2_description/meshes/Finger_Proximal.dae"/>
-      </geometry>
-      <origin xyz="0.0 0.0 0.0" rpy="0 0 1.57"/>
+<!--         <mesh filename="package://r2_description/meshes/Finger_Proximal.dae"/> -->
+         <box size="0.01 0.04 0.01" />
+      </geometry>
+      <origin xyz="0.02 0.0 0.0" rpy="0 0 1.57"/>
+<!--       <origin xyz="0.0 0.0 0.0" rpy="0 0 1.57"/> -->
     </collision>
   </link>
@@ -446,7 +466,9 @@
     <collision>
       <geometry>
-        <mesh filename="package://r2_description/meshes/Finger_Mid.dae"/>
-      </geometry>
-      <origin xyz="0.0 0.0 0.0" rpy="3.14 0 1.57"/>
+<!--         <mesh filename="package://r2_description/meshes/Finger_Mid.dae"/> -->
+        <box size="0.01 0.025 0.01" />
+      </geometry>
+<!--       <origin xyz="0.0 0.0 0.0" rpy="3.14 0 1.57"/> -->
+      <origin xyz="0.0125 0.0 0.0" rpy="3.14 0 1.57"/>
     </collision>
   </link>
@@ -472,7 +494,9 @@
     <collision>
       <geometry>
-        <mesh filename="package://r2_description/meshes/Finger_Dist.dae"/>
-      </geometry>
-      <origin xyz="0.0 0.0 0.0" rpy="0 -1.57 0"/>
+<!--         <mesh filename="package://r2_description/meshes/Finger_Dist.dae"/> -->
+        <box size="0.01 0.01 0.02" />
+      </geometry>
+<!--       <origin xyz="0.0 0.0 0.0" rpy="0 -1.57 0"/> -->
+      <origin xyz="0.015 0.0 0.0" rpy="0 -1.57 0"/>
     </collision>
   </link>
@@ -501,7 +525,9 @@
     <collision>
       <geometry>
-        <mesh filename="package://r2_description/meshes/Finger_Proximal.dae"/>
-      </geometry>
-      <origin xyz="0.0 0.0 0.0" rpy="0 0 1.57"/>
+<!--         <mesh filename="package://r2_description/meshes/Finger_Proximal.dae"/> -->
+         <box size="0.01 0.04 0.01" />
+      </geometry>
+      <origin xyz="0.02 0.0 0.0" rpy="0 0 1.57"/>
+<!--       <origin xyz="0.0 0.0 0.0" rpy="0 0 1.57"/> -->
     </collision>
   </link>
@@ -525,9 +551,11 @@
       <origin xyz="0.0 0.0 0.0" rpy="3.14 0 1.57"/>
     </visual>
-    <collision>
-      <geometry>
-        <mesh filename="package://r2_description/meshes/Finger_Mid.dae"/>
-      </geometry>
-      <origin xyz="0.0 0.0 0.0" rpy="3.14 0 1.57"/>
+   <collision>
+      <geometry>
+<!--         <mesh filename="package://r2_description/meshes/Finger_Mid.dae"/> -->
+        <box size="0.01 0.025 0.01" />
+      </geometry>
+<!--       <origin xyz="0.0 0.0 0.0" rpy="3.14 0 1.57"/> -->
+      <origin xyz="0.0125 0.0 0.0" rpy="3.14 0 1.57"/>
     </collision>
   </link>
@@ -553,7 +581,9 @@
     <collision>
       <geometry>
-        <mesh filename="package://r2_description/meshes/Finger_Dist.dae"/>
-      </geometry>
-      <origin xyz="0.0 0.0 0.0" rpy="0 -1.57 0"/>
+<!--         <mesh filename="package://r2_description/meshes/Finger_Dist.dae"/> -->
+        <box size="0.01 0.01 0.02" />
+      </geometry>
+<!--       <origin xyz="0.0 0.0 0.0" rpy="0 -1.57 0"/> -->
+      <origin xyz="0.015 0.0 0.0" rpy="0 -1.57 0"/>
     </collision>
   </link>

File: r2_description/urdf/r2.right_hand.xacro (robot description, xacro)
@@ -109,10 +109,10 @@
       <origin xyz="-0.01 0.0 0.0" rpy="-1.57 0 0"/>
     </visual>
-    <collision>
+    <!-- <collision>
       <geometry>
         <mesh filename="package://r2_description/meshes/Left_Thumb_Carp.dae" scale="0.9 0.9 0.9"/>
       </geometry>
       <origin xyz="-0.01 0.0 0.0" rpy="-1.57 0 0"/>
-    </collision>
+    </collision> -->
   </link>
   <joint name="${robot_name}right_arm/hand/thumb/joint1" type="revolute">
@@ -137,7 +137,9 @@
     <collision>
       <geometry>
-        <mesh filename="package://r2_description/meshes/Right_Thumb_MtCar.dae" scale="0.9 0.9 0.9"/>
-      </geometry>
-      <origin xyz="-0.0 0 0.0" rpy="-1.57 -1.57 0 "/>
+ <!--        <mesh filename="package://r2_description/meshes/Left_Thumb_MtCar.dae"/> -->
+        <box size="0.01 0.02 0.01" />
+      </geometry>
+<!--       <origin xyz="0.0 0.0 0.0" rpy="-1.57 -1.57 0"/> -->
+      <origin xyz="0.02 0.0 0.0" rpy="-1.57 -1.57 0"/>
     </collision>
   </link>
@@ -163,7 +165,9 @@
     <collision>
       <geometry>
-        <mesh filename="package://r2_description/meshes/Thumb_Proximal.dae"/>
-      </geometry>
-      <origin xyz="0.0 0.0 0.0" rpy="3.14 0 1.57"/>
+<!--         <mesh filename="package://r2_description/meshes/Thumb_Proximal.dae"/> -->
+          <box size="0.01 0.03 0.01" />
+      </geometry>
+<!--       <origin xyz="0.0 0.0 0.0" rpy="3.14 0 1.57"/> -->
+      <origin xyz="0.022 0.0 0.0" rpy="3.14 0 1.57"/>
     </collision>
   </link>
@@ -189,7 +193,9 @@
     <collision>
       <geometry>
-        <mesh filename="package://r2_description/meshes/Thumb_Dist.dae"/>
-      </geometry>
-      <origin xyz="0.0 0.0 0.0" rpy="3.14 3.14 0"/>
+<!--         <mesh filename="package://r2_description/meshes/Thumb_Dist.dae"/> -->
+        <box size="0.025 0.01 0.01" />
+      </geometry>
+ <!--      <origin xyz="0.0 0.0 0.0" rpy="3.14 3.14 0"/> -->
+      <origin xyz="0.015 0.0 0.0" rpy="3.14 3.14 0"/>
     </collision>
   </link>
@@ -238,7 +244,9 @@
     <collision>
       <geometry>
-        <mesh filename="package://r2_description/meshes/Finger_Proximal.dae"/>
-      </geometry>
-      <origin xyz="0.0 0.0 0.0" rpy="0 0 1.57"/>
+<!--         <mesh filename="package://r2_description/meshes/Finger_Proximal.dae"/> -->
+         <box size="0.01 0.04 0.01" />
+      </geometry>
+      <origin xyz="0.02 0.0 0.0" rpy="0 0 1.57"/>
+<!--       <origin xyz="0.0 0.0 0.0" rpy="0 0 1.57"/> -->
     </collision>
   </link>
@@ -264,7 +272,9 @@
     <collision>
       <geometry>
-        <mesh filename="package://r2_description/meshes/Finger_Mid.dae"/>
-      </geometry>
-      <origin xyz="0.0 0.0 0.0" rpy="3.14 0 1.57"/>
+<!--         <mesh filename="package://r2_description/meshes/Finger_Mid.dae"/> -->
+        <box size="0.01 0.025 0.01" />
+      </geometry>
+<!--       <origin xyz="0.0 0.0 0.0" rpy="3.14 0 1.57"/> -->
+      <origin xyz="0.0125 0.0 0.0" rpy="3.14 0 1.57"/>
     </collision>
   </link>
@@ -290,7 +300,9 @@
     <collision>
       <geometry>
-        <mesh filename="package://r2_description/meshes/Finger_Dist.dae"/>
-      </geometry>
-      <origin xyz="0.0 0.0 0.0" rpy="0 -1.57 0"/>
+<!--         <mesh filename="package://r2_description/meshes/Finger_Dist.dae"/> -->
+        <box size="0.01 0.01 0.02" />
+      </geometry>
+<!--       <origin xyz="0.0 0.0 0.0" rpy="0 -1.57 0"/> -->
+      <origin xyz="0.015 0.0 0.0" rpy="0 -1.57 0"/>
     </collision>
   </link>
@@ -339,7 +351,9 @@
     <collision>
       <geometry>
-        <mesh filename="package://r2_description/meshes/Finger_Proximal.dae" scale="0.9 0.9 0.9"/>
-      </geometry>
-      <origin xyz="0.0 0.0 0.0" rpy="0 0 1.57"/>
+<!--         <mesh filename="package://r2_description/meshes/Finger_Proximal.dae"/> -->
+         <box size="0.01 0.04 0.01" />
+      </geometry>
+      <origin xyz="0.02 0.0 0.0" rpy="0 0 1.57"/>
+<!--       <origin xyz="0.0 0.0 0.0" rpy="0 0 1.57"/> -->
     </collision>
   </link>
@@ -365,7 +379,9 @@
     <collision>
       <geometry>
-        <mesh filename="package://r2_description/meshes/Finger_Mid.dae" scale="0.9 0.9 0.9"/>
-      </geometry>
-      <origin xyz="0.0 0.0 0.0" rpy="3.14 0 1.57"/>
+<!--         <mesh filename="package://r2_description/meshes/Finger_Mid.dae"/> -->
+        <box size="0.01 0.025 0.01" />
+      </geometry>
+<!--       <origin xyz="0.0 0.0 0.0" rpy="3.14 0 1.57"/> -->
+      <origin xyz="0.0125 0.0 0.0" rpy="3.14 0 1.57"/>
     </collision>
   </link>
@@ -391,7 +407,9 @@
     <collision>
       <geometry>
-        <mesh filename="package://r2_description/meshes/Finger_Dist.dae" scale="0.9 0.9 0.9"/>
-      </geometry>
-      <origin xyz="0.0 0.0 0.0" rpy="0 -1.57 0"/>
+<!--         <mesh filename="package://r2_description/meshes/Finger_Dist.dae"/> -->
+        <box size="0.01 0.01 0.02" />
+      </geometry>
+<!--       <origin xyz="0.0 0.0 0.0" rpy="0 -1.57 0"/> -->
+      <origin xyz="0.015 0.0 0.0" rpy="0 -1.57 0"/>
     </collision>
   </link>
@@ -420,7 +438,9 @@
     <collision>
       <geometry>
-        <mesh filename="package://r2_description/meshes/Finger_Proximal.dae" scale="0.9 0.9 0.9"/>
-      </geometry>
-      <origin xyz="0.0 0.0 0.0" rpy="0 0 1.57"/>
+<!--         <mesh filename="package://r2_description/meshes/Finger_Proximal.dae"/> -->
+         <box size="0.01 0.04 0.01" />
+      </geometry>
+      <origin xyz="0.02 0.0 0.0" rpy="0 0 1.57"/>
+<!--       <origin xyz="0.0 0.0 0.0" rpy="0 0 1.57"/> -->
     </collision>
   </link>
@@ -446,7 +466,9 @@
     <collision>
       <geometry>
-        <mesh filename="package://r2_description/meshes/Finger_Mid.dae" scale="0.9 0.9 0.9"/>
-      </geometry>
-      <origin xyz="0.0 0.0 0.0" rpy="3.14 0 1.57"/>
+<!--         <mesh filename="package://r2_description/meshes/Finger_Mid.dae"/> -->
+        <box size="0.01 0.025 0.01" />
+      </geometry>
+<!--       <origin xyz="0.0 0.0 0.0" rpy="3.14 0 1.57"/> -->
+      <origin xyz="0.0125 0.0 0.0" rpy="3.14 0 1.57"/>
     </collision>
   </link>
@@ -472,7 +494,9 @@
     <collision>
       <geometry>
-        <mesh filename="package://r2_description/meshes/Finger_Dist.dae" scale="0.9 0.9 0.9"/>
-      </geometry>
-      <origin xyz="0.0 0.0 0.0" rpy="0 -1.57 0"/>
+<!--         <mesh filename="package://r2_description/meshes/Finger_Dist.dae"/> -->
+        <box size="0.01 0.01 0.02" />
+      </geometry>
+<!--       <origin xyz="0.0 0.0 0.0" rpy="0 -1.57 0"/> -->
+      <origin xyz="0.015 0.0 0.0" rpy="0 -1.57 0"/>
     </collision>
   </link>
@@ -501,7 +525,9 @@
     <collision>
       <geometry>
-        <mesh filename="package://r2_description/meshes/Finger_Proximal.dae" scale="0.9 0.9 0.9"/>
-      </geometry>
-      <origin xyz="0.0 0.0 0.0" rpy="0 0 1.57"/>
+<!--         <mesh filename="package://r2_description/meshes/Finger_Proximal.dae"/> -->
+         <box size="0.01 0.04 0.01" />
+      </geometry>
+      <origin xyz="0.02 0.0 0.0" rpy="0 0 1.57"/>
+<!--       <origin xyz="0.0 0.0 0.0" rpy="0 0 1.57"/> -->
     </collision>
   </link>
@@ -527,7 +553,9 @@
     <collision>
       <geometry>
-        <mesh filename="package://r2_description/meshes/Finger_Mid.dae" scale="0.9 0.9 0.9"/>
-      </geometry>
-      <origin xyz="0.0 0.0 0.0" rpy="3.14 0 1.57"/>
+<!--         <mesh filename="package://r2_description/meshes/Finger_Mid.dae"/> -->
+        <box size="0.01 0.025 0.01" />
+      </geometry>
+<!--       <origin xyz="0.0 0.0 0.0" rpy="3.14 0 1.57"/> -->
+      <origin xyz="0.0125 0.0 0.0" rpy="3.14 0 1.57"/>
     </collision>
   </link>
@@ -553,7 +581,9 @@
     <collision>
       <geometry>
-        <mesh filename="package://r2_description/meshes/Finger_Dist.dae" scale="0.9 0.9 0.9"/>
-      </geometry>
-      <origin xyz="0.0 0.0 0.0" rpy="0 -1.57 0"/>
+<!--         <mesh filename="package://r2_description/meshes/Finger_Dist.dae"/> -->
+        <box size="0.01 0.01 0.02" />
+      </geometry>
+<!--       <origin xyz="0.0 0.0 0.0" rpy="0 -1.57 0"/> -->
+      <origin xyz="0.015 0.0 0.0" rpy="0 -1.57 0"/>
     </collision>
   </link>
