Commit message: updated joint names

File: r2_description/urdf/r2.left_arm.xacro (robot description, xacro)
@@ -155,5 +155,5 @@
     </inertial>
   </link>
-  <joint name="${robot_name}left_arm/joint5" type="revolute">
+  <joint name="${robot_name}left_arm/wrist/pitch" type="revolute">
     <parent link="${robot_name}left_lower_arm"/>
     <child link="${robot_name}left_wrist_pitch"/>
@@ -170,5 +170,5 @@
     </inertial>
   </link>
-  <joint name="${robot_name}left_arm/joint6" type="revolute">
+  <joint name="${robot_name}left_arm/wrist/yaw" type="revolute">
     <parent link="${robot_name}left_wrist_pitch"/>
     <child link="${robot_name}left_wrist_yaw"/>

File: r2_description/urdf/r2.left_hand.xacro (robot description, xacro)
@@ -37,5 +37,5 @@
   <property name="left_arm_hand_little_j2_damping" value= "0.1" />
   <property name="left_arm_hand_little_j2_friction" value= "0.0" />
-  <joint name="${robot_name}left_arm/hand/thumb/joint0" type="revolute">
+  <joint name="${robot_name}left_arm/hand/thumb/roll" type="revolute">
     <parent link="${robot_name}left_wrist_yaw"/>
     <child link="${robot_name}left_thumb_base"/>
@@ -50,5 +50,5 @@
     <origin xyz=" 0.0994646728 0.0271119346 -0.0161544 " rpy=" 0.0 -0.0 0.122172725275 " />
   </joint>
-  <joint name="${robot_name}left_arm/hand/index/joint0" type="revolute">
+  <joint name="${robot_name}left_arm/hand/index/yaw" type="revolute">
     <parent link="${robot_name}left_index_base"/>
     <child link="${robot_name}left_index_yaw"/>
@@ -63,5 +63,5 @@
     <origin xyz=" 0.10646537 0.00254 -0.0161544 " rpy=" 0.0 -0.0 0.0 " />
   </joint>
-  <joint name="${robot_name}left_arm/hand/middle/joint0" type="revolute">
+  <joint name="${robot_name}left_arm/hand/middle/yaw" type="revolute">
     <parent link="${robot_name}left_middle_base"/>
     <child link="${robot_name}left_middle_yaw"/>
@@ -71,5 +71,5 @@
     <dynamics damping="${left_arm_hand_middle_j0_damping}" friction="${left_arm_hand_middle_j0_friction}"/>
   </joint>
-  <joint name="${robot_name}left_arm/hand/ring/joint0" type="revolute">
+  <joint name="${robot_name}left_arm/hand/ring/proximal" type="revolute">
     <parent link="${robot_name}left_wrist_yaw"/>
     <child link="${robot_name}left_ring_proximal"/>
@@ -79,5 +79,5 @@
     <dynamics damping="${left_arm_hand_ring_j0_damping}" friction="${left_arm_hand_ring_j0_friction}"/>
   </joint>
-  <joint name="${robot_name}left_arm/hand/little/joint0" type="revolute">
+  <joint name="${robot_name}left_arm/hand/little/proximal" type="revolute">
     <parent link="${robot_name}left_wrist_yaw"/>
     <child link="${robot_name}left_little_proximal"/>
@@ -116,5 +116,5 @@
     </collision>
   </link>
-  <joint name="${robot_name}left_arm/hand/thumb/joint1" type="revolute">
+  <joint name="${robot_name}left_arm/hand/thumb/proximal" type="revolute">
     <parent link="${robot_name}left_thumb_proximal"/>
     <child link="${robot_name}left_thumb_medial_prime"/>
@@ -142,5 +142,5 @@
     </collision>
   </link>
-  <joint name="${robot_name}left_arm/hand/thumb/joint2" type="revolute">
+  <joint name="${robot_name}left_arm/hand/thumb/medial" type="revolute">
     <parent link="${robot_name}left_thumb_medial_prime"/>
     <child link="${robot_name}left_thumb_medial"/>
@@ -168,5 +168,5 @@
     </collision>
   </link>
-  <joint name="${robot_name}left_arm/hand/thumb/joint3" type="revolute">
+  <joint name="${robot_name}left_arm/hand/thumb/distal" type="revolute">
     <parent link="${robot_name}left_thumb_medial"/>
     <child link="${robot_name}left_thumb_distal"/>
@@ -217,5 +217,5 @@
     </inertial>
   </link>
-  <joint name="${robot_name}left_arm/hand/index/joint1" type="revolute">
+  <joint name="${robot_name}left_arm/hand/index/proximal" type="revolute">
     <parent link="${robot_name}left_index_yaw"/>
     <child link="${robot_name}left_index_proximal"/>
@@ -243,5 +243,5 @@
     </collision>
   </link>
-  <joint name="${robot_name}left_arm/hand/index/joint2" type="revolute">
+  <joint name="${robot_name}left_arm/hand/index/medial" type="revolute">
     <parent link="${robot_name}left_index_proximal"/>
     <child link="${robot_name}left_index_medial"/>
@@ -269,5 +269,5 @@
     </collision>
   </link>
-  <joint name="${robot_name}left_arm/hand/index/joint3" type="revolute">
+  <joint name="${robot_name}left_arm/hand/index/distal" type="revolute">
     <parent link="${robot_name}left_index_medial"/>
     <child link="${robot_name}left_index_distal"/>
@@ -318,5 +318,5 @@
     </inertial>
   </link>
-  <joint name="${robot_name}left_arm/hand/middle/joint1" type="revolute">
+  <joint name="${robot_name}left_arm/hand/middle/proximal" type="revolute">
     <parent link="${robot_name}left_middle_yaw"/>
     <child link="${robot_name}left_middle_proximal"/>
@@ -344,5 +344,5 @@
     </collision>
   </link>
-  <joint name="${robot_name}left_arm/hand/middle/joint2" type="revolute">
+  <joint name="${robot_name}left_arm/hand/middle/medial" type="revolute">
     <parent link="${robot_name}left_middle_proximal"/>
     <child link="${robot_name}left_middle_medial"/>
@@ -370,5 +370,5 @@
     </collision>
   </link>
-  <joint name="${robot_name}left_arm/hand/middle/joint3" type="revolute">
+  <joint name="${robot_name}left_arm/hand/middle/distal" type="revolute">
     <parent link="${robot_name}left_middle_medial"/>
     <child link="${robot_name}left_middle_distal"/>
@@ -425,5 +425,5 @@
     </collision>
   </link>
-  <joint name="${robot_name}left_arm/hand/ring/joint1" type="revolute">
+  <joint name="${robot_name}left_arm/hand/ring/medial" type="revolute">
     <parent link="${robot_name}left_ring_proximal"/>
     <child link="${robot_name}left_ring_medial"/>
@@ -451,5 +451,5 @@
     </collision>
   </link>
-  <joint name="${robot_name}left_arm/hand/ring/joint2" type="revolute">
+  <joint name="${robot_name}left_arm/hand/ring/distal" type="revolute">
     <parent link="${robot_name}left_ring_medial"/>
     <child link="${robot_name}left_ring_distal"/>
@@ -506,5 +506,5 @@
     </collision>
   </link>
-  <joint name="${robot_name}left_arm/hand/little/joint1" type="revolute">
+  <joint name="${robot_name}left_arm/hand/little/medial" type="revolute">
     <parent link="${robot_name}left_little_proximal"/>
     <child link="${robot_name}left_little_medial"/>
@@ -532,5 +532,5 @@
     </collision>
   </link>
-  <joint name="${robot_name}left_arm/hand/little/joint2" type="revolute">
+  <joint name="${robot_name}left_arm/hand/little/distal" type="revolute">
     <parent link="${robot_name}left_little_medial"/>
     <child link="${robot_name}left_little_distal"/>

File: r2_description/urdf/r2.right_arm.xacro (robot description, xacro)
@@ -155,5 +155,5 @@
     </inertial>
   </link>
-  <joint name="${robot_name}right_arm/joint5" type="revolute">
+  <joint name="${robot_name}right_arm/wrist/pitch" type="revolute">
     <parent link="${robot_name}right_lower_arm"/>
     <child link="${robot_name}right_wrist_pitch"/>
@@ -170,5 +170,5 @@
     </inertial>
   </link>
-  <joint name="${robot_name}right_arm/joint6" type="revolute">
+  <joint name="${robot_name}right_arm/wrist/yaw" type="revolute">
     <parent link="${robot_name}right_wrist_pitch"/>
     <child link="${robot_name}right_wrist_yaw"/>

File: r2_description/urdf/r2.right_hand.xacro (robot description, xacro)
@@ -37,5 +37,5 @@
   <property name="right_arm_hand_little_j2_damping" value= "0.1" />
   <property name="right_arm_hand_little_j2_friction" value= "0.0" />
-<joint name="${robot_name}right_arm/hand/thumb/joint0" type="revolute">
+<joint name="${robot_name}right_arm/hand/thumb/roll" type="revolute">
     <parent link="${robot_name}right_wrist_yaw"/>
     <child link="${robot_name}right_thumb_base"/>
@@ -50,5 +50,5 @@
     <origin xyz=" 0.0994646728 -0.0271119346 -0.0161544 " rpy=" 0.0 -0.0 -0.122172725275  " />
   </joint>
-  <joint name="${robot_name}right_arm/hand/index/joint0" type="revolute">
+  <joint name="${robot_name}right_arm/hand/index/yaw" type="revolute">
     <parent link="${robot_name}right_index_base"/>
     <child link="${robot_name}right_index_yaw"/>
@@ -63,5 +63,5 @@
     <origin xyz="0.10646537 -0.00254 -0.0161544 " rpy=" 0.0 -0.0 0.0 " />
   </joint>
-  <joint name="${robot_name}right_arm/hand/middle/joint0" type="revolute">
+  <joint name="${robot_name}right_arm/hand/middle/yaw" type="revolute">
     <parent link="${robot_name}right_middle_base"/>
     <child link="${robot_name}right_middle_yaw"/>
@@ -71,5 +71,5 @@
     <dynamics damping="${right_arm_hand_middle_j0_damping}" friction="${right_arm_hand_middle_j0_friction}"/>
   </joint>
-  <joint name="${robot_name}right_arm/hand/ring/joint0" type="revolute">
+  <joint name="${robot_name}right_arm/hand/ring/proximal" type="revolute">
     <parent link="${robot_name}right_wrist_yaw"/>
     <child link="${robot_name}right_ring_proximal"/>
@@ -79,5 +79,5 @@
     <dynamics damping="${right_arm_hand_ring_j0_damping}" friction="${right_arm_hand_ring_j0_friction}"/>
   </joint>
-  <joint name="${robot_name}right_arm/hand/little/joint0" type="revolute">
+  <joint name="${robot_name}right_arm/hand/little/proximal" type="revolute">
     <parent link="${robot_name}right_wrist_yaw"/>
     <child link="${robot_name}right_little_proximal"/>
@@ -116,5 +116,5 @@
     </collision>
   </link>
-  <joint name="${robot_name}right_arm/hand/thumb/joint1" type="revolute">
+  <joint name="${robot_name}right_arm/hand/thumb/proximal" type="revolute">
     <parent link="${robot_name}right_thumb_proximal"/>
     <child link="${robot_name}right_thumb_medial_prime"/>
@@ -142,5 +142,5 @@
     </collision>
   </link>
-  <joint name="${robot_name}right_arm/hand/thumb/joint2" type="revolute">
+  <joint name="${robot_name}right_arm/hand/thumb/medial" type="revolute">
     <parent link="${robot_name}right_thumb_medial_prime"/>
     <child link="${robot_name}right_thumb_medial"/>
@@ -168,5 +168,5 @@
     </collision>
   </link>
-  <joint name="${robot_name}right_arm/hand/thumb/joint3" type="revolute">
+  <joint name="${robot_name}right_arm/hand/thumb/distal" type="revolute">
     <parent link="${robot_name}right_thumb_medial"/>
     <child link="${robot_name}right_thumb_distal"/>
@@ -217,5 +217,5 @@
     </inertial>
   </link>
-  <joint name="${robot_name}right_arm/hand/index/joint1" type="revolute">
+  <joint name="${robot_name}right_arm/hand/index/proximal" type="revolute">
     <parent link="${robot_name}right_index_yaw"/>
     <child link="${robot_name}right_index_proximal"/>
@@ -243,5 +243,5 @@
     </collision>
   </link>
-  <joint name="${robot_name}right_arm/hand/index/joint2" type="revolute">
+  <joint name="${robot_name}right_arm/hand/index/medial" type="revolute">
     <parent link="${robot_name}right_index_proximal"/>
     <child link="${robot_name}right_index_medial"/>
@@ -269,5 +269,5 @@
     </collision>
   </link>
-  <joint name="${robot_name}right_arm/hand/index/joint3" type="revolute">
+  <joint name="${robot_name}right_arm/hand/index/distal" type="revolute">
     <parent link="${robot_name}right_index_medial"/>
     <child link="${robot_name}right_index_distal"/>
@@ -318,5 +318,5 @@
     </inertial>
   </link>
-  <joint name="${robot_name}right_arm/hand/middle/joint1" type="revolute">
+  <joint name="${robot_name}right_arm/hand/middle/proximal" type="revolute">
     <parent link="${robot_name}right_middle_yaw"/>
     <child link="${robot_name}right_middle_proximal"/>
@@ -344,5 +344,5 @@
     </collision>
   </link>
-  <joint name="${robot_name}right_arm/hand/middle/joint2" type="revolute">
+  <joint name="${robot_name}right_arm/hand/middle/medial" type="revolute">
     <parent link="${robot_name}right_middle_proximal"/>
     <child link="${robot_name}right_middle_medial"/>
@@ -370,5 +370,5 @@
     </collision>
   </link>
-  <joint name="${robot_name}right_arm/hand/middle/joint3" type="revolute">
+  <joint name="${robot_name}right_arm/hand/middle/distal" type="revolute">
     <parent link="${robot_name}right_middle_medial"/>
     <child link="${robot_name}right_middle_distal"/>
@@ -425,5 +425,5 @@
     </collision>
   </link>
-  <joint name="${robot_name}right_arm/hand/ring/joint1" type="revolute">
+  <joint name="${robot_name}right_arm/hand/ring/medial" type="revolute">
     <parent link="${robot_name}right_ring_proximal"/>
     <child link="${robot_name}right_ring_medial"/>
@@ -451,5 +451,5 @@
     </collision>
   </link>
-  <joint name="${robot_name}right_arm/hand/ring/joint2" type="revolute">
+  <joint name="${robot_name}right_arm/hand/ring/distal" type="revolute">
     <parent link="${robot_name}right_ring_medial"/>
     <child link="${robot_name}right_ring_distal"/>
@@ -506,5 +506,5 @@
     </collision>
   </link>
-  <joint name="${robot_name}right_arm/hand/little/joint1" type="revolute">
+  <joint name="${robot_name}right_arm/hand/little/medial" type="revolute">
     <parent link="${robot_name}right_little_proximal"/>
     <child link="${robot_name}right_little_medial"/>
@@ -532,5 +532,5 @@
     </collision>
   </link>
-  <joint name="${robot_name}right_arm/hand/little/joint2" type="revolute">
+  <joint name="${robot_name}right_arm/hand/little/distal" type="revolute">
     <parent link="${robot_name}right_little_medial"/>
     <child link="${robot_name}right_little_distal"/>
