Commit message: making left and right arm, hand more symmetric

File: r2_description/urdf/r2.left_arm.xacro (robot description, xacro)
@@ -89,5 +89,5 @@
     <collision>
       <geometry>
-        <mesh filename="package://r2_description/meshes/Left_Upper_Arm.dae" scale="0.8 0.8 0.8"/>
+        <mesh filename="package://r2_description/meshes/Left_Upper_Arm.dae" />
       </geometry>
       <origin rpy="0 0 3.14" xyz="0 0 .1016"/>

File: r2_description/urdf/r2.right_arm.xacro (robot description, xacro)
@@ -140,6 +140,6 @@
         <mesh filename="package://r2_description/meshes/Right_Forearm.dae"/>
       </geometry>
-      <material name="dirty_white"/>
-      <origin xyz="0 0 0.1"/>
+	  <origin xyz="0 0 0.1"/>
+      <material name="dirty_white"/>
     </visual>
     <collision>
@@ -188,5 +188,5 @@
     <parent link="${robot_name}right_wrist_yaw"/>
     <child link="${robot_name}right_palm"/>
-    <origin rpy=" 0.0 -0.0 0.0299" xyz=" 0.0 0.0 0.0"/>
+    <origin rpy=" 0.0 -0.0 0.014" xyz=" 0.0 0.0 0.0"/>
   </joint>
   <link name="${robot_name}right_palm">
@@ -204,4 +204,5 @@
     </collision>
     <inertial>
+		<origin xyz="0.067564   -0.0253746   -0.00090932"/>
         <mass value="1.1"/>
         <inertia ixx="0.1"  ixy="0.0"  ixz="0.0"  iyy="0.1"  iyz="0.0"  izz="0.1"/>

File: r2_description/urdf/r2.right_hand.xacro (robot description, xacro)
@@ -40,5 +40,5 @@
     <parent link="${robot_name}right_wrist_yaw"/>
     <child link="${robot_name}right_thumb_base"/>
-    <origin xyz="0.03302 -0.03048 0.00635 " rpy=" 1.57079632679 0.174532791018 -1.30899687745 " />
+    <origin xyz="0.03302 -0.03048 0.00635 " rpy=" 1.57079632679 0.0 -1.30899687745 " />
     <axis xyz="0 0 1"/>
     <limit effort="10000000.0" lower="0.0" upper="1.2217" velocity="1000"/>
@@ -82,5 +82,5 @@
     <parent link="${robot_name}right_wrist_yaw"/>
     <child link="${robot_name}right_little_proximal"/>
-    <origin xyz=" 0.094635701 0.0403792436 -0.0060878212 " rpy=" 1.53588943985 -0.0872667473393 0.17453258148  " />
+    <origin xyz=" 0.094635701 0.0403792436 -0.0060878212 " rpy=" 1.60570321374 -0.0872667473393 0.17453258148  " />
     <axis xyz="0 0 1"/>
     <limit effort="10000000.0" lower="0" upper="2.9671" velocity="1000"/>
@@ -100,5 +100,5 @@
   <link name="${robot_name}right_thumb_proximal">
     <inertial>
-      <mass value=".05"/>
+      <mass value=".001"/>
       <inertia ixx=".0010" ixy="0.0" ixz="0.0" iyy=".0010" iyz="0.0" izz=".0010"/>
     </inertial>
@@ -126,5 +126,5 @@
   <link name="${robot_name}right_thumb_medial_prime">
     <inertial>
-      <mass value=".05"/>
+      <mass value=".001"/>
       <inertia ixx=".0010" ixy="0.0" ixz="0.0" iyy=".0010" iyz="0.0" izz=".0010"/>
     </inertial>
@@ -152,5 +152,5 @@
   <link name="${robot_name}right_thumb_medial">
     <inertial>
-      <mass value=".05"/>
+      <mass value=".001"/>
       <inertia ixx=".0010" ixy="0.0" ixz="0.0" iyy=".0010" iyz="0.0" izz=".0010"/>
     </inertial>
@@ -178,5 +178,5 @@
   <link name="${robot_name}right_thumb_distal">
     <inertial>
-      <mass value=".05"/>
+      <mass value=".001"/>
       <inertia ixx=".0010" ixy="0.0" ixz="0.0" iyy=".0010" iyz="0.0" izz=".0010"/>
     </inertial>
@@ -201,17 +201,17 @@
   <link name="${robot_name}right_thumb_tip">
     <inertial>
+      <mass value=".001"/>
+      <inertia ixx=".0010" ixy="0.0" ixz="0.0" iyy=".0010" iyz="0.0" izz=".0010"/>
+    </inertial>
+  </link>
+  <link name="${robot_name}right_index_base">
+    <inertial>
       <mass value=".05"/>
       <inertia ixx=".0010" ixy="0.0" ixz="0.0" iyy=".0010" iyz="0.0" izz=".0010"/>
     </inertial>
   </link>
-  <link name="${robot_name}right_index_base">
-    <inertial>
-      <mass value=".05"/>
-      <inertia ixx=".0010" ixy="0.0" ixz="0.0" iyy=".0010" iyz="0.0" izz=".0010"/>
-    </inertial>
-  </link>
   <link name="${robot_name}right_index_yaw">
     <inertial>
-      <mass value=".05"/>
+      <mass value=".001"/>
       <inertia ixx=".0010" ixy="0.0" ixz="0.0" iyy=".0010" iyz="0.0" izz=".0010"/>
     </inertial>
@@ -227,5 +227,5 @@
   <link name="${robot_name}right_index_proximal">
     <inertial>
-      <mass value=".05"/>
+      <mass value=".001"/>
       <inertia ixx=".0010" ixy="0.0" ixz="0.0" iyy=".0010" iyz="0.0" izz=".0010"/>
     </inertial>
@@ -253,5 +253,5 @@
   <link name="${robot_name}right_index_medial">
     <inertial>
-      <mass value=".05"/>
+      <mass value=".001"/>
       <inertia ixx=".0010" ixy="0.0" ixz="0.0" iyy=".0010" iyz="0.0" izz=".0010"/>
     </inertial>
@@ -279,5 +279,5 @@
   <link name="${robot_name}right_index_distal">
     <inertial>
-      <mass value=".05"/>
+      <mass value=".001"/>
       <inertia ixx=".0010" ixy="0.0" ixz="0.0" iyy=".0010" iyz="0.0" izz=".0010"/>
     </inertial>
@@ -302,5 +302,5 @@
   <link name="${robot_name}right_index_tip">
     <inertial>
-      <mass value=".05"/>
+      <mass value=".001"/>
       <inertia ixx=".0010" ixy="0.0" ixz="0.0" iyy=".0010" iyz="0.0" izz=".0010"/>
     </inertial>
@@ -328,16 +328,16 @@
   <link name="${robot_name}right_middle_proximal">
     <inertial>
-      <mass value=".05"/>
-      <inertia ixx=".0010" ixy="0.0" ixz="0.0" iyy=".0010" iyz="0.0" izz=".0010"/>
-    </inertial>
-    <visual>
-      <geometry>
-        <mesh filename="package://r2_description/meshes/Finger_Proximal.dae"/>
-      </geometry>
-      <origin xyz="0.0 0.0 0.0" rpy="0 0 1.57"/>
-    </visual>
-    <collision>
-      <geometry>
-        <mesh filename="package://r2_description/meshes/Finger_Proximal.dae" scale="0.9 0.9 0.9"/>
+      <mass value=".001"/>
+      <inertia ixx=".0010" ixy="0.0" ixz="0.0" iyy=".0010" iyz="0.0" izz=".0010"/>
+    </inertial>
+    <visual>
+      <geometry>
+        <mesh filename="package://r2_description/meshes/Finger_Proximal.dae"/>
+      </geometry>
+      <origin xyz="0.0 0.0 0.0" rpy="0 0 1.57"/>
+    </visual>
+    <collision>
+      <geometry>
+        <mesh filename="package://r2_description/meshes/Finger_Proximal.dae"/>
       </geometry>
       <origin xyz="0.0 0.0 0.0" rpy="0 0 1.57"/>
@@ -354,16 +354,16 @@
   <link name="${robot_name}right_middle_medial">
     <inertial>
-      <mass value=".05"/>
-      <inertia ixx=".0010" ixy="0.0" ixz="0.0" iyy=".0010" iyz="0.0" izz=".0010"/>
-    </inertial>
-    <visual>
-      <geometry>
-        <mesh filename="package://r2_description/meshes/Finger_Mid.dae"/>
-      </geometry>
-      <origin xyz="0.0 0.0 0.0" rpy="3.14 0 1.57"/>
-    </visual>
-    <collision>
-      <geometry>
-        <mesh filename="package://r2_description/meshes/Finger_Mid.dae" scale="0.9 0.9 0.9"/>
+      <mass value=".001"/>
+      <inertia ixx=".0010" ixy="0.0" ixz="0.0" iyy=".0010" iyz="0.0" izz=".0010"/>
+    </inertial>
+    <visual>
+      <geometry>
+        <mesh filename="package://r2_description/meshes/Finger_Mid.dae"/>
+      </geometry>
+      <origin xyz="0.0 0.0 0.0" rpy="3.14 0 1.57"/>
+    </visual>
+    <collision>
+      <geometry>
+        <mesh filename="package://r2_description/meshes/Finger_Mid.dae"/>
       </geometry>
       <origin xyz="0.0 0.0 0.0" rpy="3.14 0 1.57"/>
@@ -380,16 +380,16 @@
   <link name="${robot_name}right_middle_distal">
     <inertial>
-      <mass value=".05"/>
-      <inertia ixx=".0010" ixy="0.0" ixz="0.0" iyy=".0010" iyz="0.0" izz=".0010"/>
-    </inertial>
-    <visual>
-      <geometry>
-        <mesh filename="package://r2_description/meshes/Finger_Dist.dae"/>
-      </geometry>
-      <origin xyz="0.0 0.0 0.0" rpy="0 -1.57 0"/>
-    </visual>
-    <collision>
-      <geometry>
-        <mesh filename="package://r2_description/meshes/Finger_Dist.dae" scale="0.9 0.9 0.9"/>
+      <mass value=".001"/>
+      <inertia ixx=".0010" ixy="0.0" ixz="0.0" iyy=".0010" iyz="0.0" izz=".0010"/>
+    </inertial>
+    <visual>
+      <geometry>
+        <mesh filename="package://r2_description/meshes/Finger_Dist.dae"/>
+      </geometry>
+      <origin xyz="0.0 0.0 0.0" rpy="0 -1.57 0"/>
+    </visual>
+    <collision>
+      <geometry>
+        <mesh filename="package://r2_description/meshes/Finger_Dist.dae"/>
       </geometry>
       <origin xyz="0.0 0.0 0.0" rpy="0 -1.57 0"/>
@@ -403,5 +403,5 @@
   <link name="${robot_name}right_middle_tip">
     <inertial>
-      <mass value=".05"/>
+      <mass value=".001"/>
       <inertia ixx=".0010" ixy="0.0" ixz="0.0" iyy=".0010" iyz="0.0" izz=".0010"/>
     </inertial>
@@ -409,16 +409,16 @@
   <link name="${robot_name}right_ring_proximal">
     <inertial>
-      <mass value=".05"/>
-      <inertia ixx=".0010" ixy="0.0" ixz="0.0" iyy=".0010" iyz="0.0" izz=".0010"/>
-    </inertial>
-    <visual>
-      <geometry>
-        <mesh filename="package://r2_description/meshes/Finger_Proximal.dae"/>
-      </geometry>
-      <origin xyz="0.0 0.0 0.0" rpy="0 0 1.57"/>
-    </visual>
-    <collision>
-      <geometry>
-        <mesh filename="package://r2_description/meshes/Finger_Proximal.dae" scale="0.9 0.9 0.9"/>
+      <mass value=".001"/>
+      <inertia ixx=".0010" ixy="0.0" ixz="0.0" iyy=".0010" iyz="0.0" izz=".0010"/>
+    </inertial>
+    <visual>
+      <geometry>
+        <mesh filename="package://r2_description/meshes/Finger_Proximal.dae"/>
+      </geometry>
+      <origin xyz="0.0 0.0 0.0" rpy="0 0 1.57"/>
+    </visual>
+    <collision>
+      <geometry>
+        <mesh filename="package://r2_description/meshes/Finger_Proximal.dae"/>
       </geometry>
       <origin xyz="0.0 0.0 0.0" rpy="0 0 1.57"/>
@@ -435,16 +435,16 @@
   <link name="${robot_name}right_ring_medial">
     <inertial>
-      <mass value=".05"/>
-      <inertia ixx=".0010" ixy="0.0" ixz="0.0" iyy=".0010" iyz="0.0" izz=".0010"/>
-    </inertial>
-    <visual>
-      <geometry>
-        <mesh filename="package://r2_description/meshes/Finger_Mid.dae"/>
-      </geometry>
-      <origin xyz="0.0 0.0 0.0" rpy="3.14 0 1.57"/>
-    </visual>
-    <collision>
-      <geometry>
-        <mesh filename="package://r2_description/meshes/Finger_Mid.dae" scale="0.9 0.9 0.9"/>
+      <mass value=".001"/>
+      <inertia ixx=".0010" ixy="0.0" ixz="0.0" iyy=".0010" iyz="0.0" izz=".0010"/>
+    </inertial>
+    <visual>
+      <geometry>
+        <mesh filename="package://r2_description/meshes/Finger_Mid.dae"/>
+      </geometry>
+      <origin xyz="0.0 0.0 0.0" rpy="3.14 0 1.57"/>
+    </visual>
+    <collision>
+      <geometry>
+        <mesh filename="package://r2_description/meshes/Finger_Mid.dae"/>
       </geometry>
       <origin xyz="0.0 0.0 0.0" rpy="3.14 0 1.57"/>
@@ -461,16 +461,16 @@
   <link name="${robot_name}right_ring_distal">
     <inertial>
-      <mass value=".05"/>
-      <inertia ixx=".0010" ixy="0.0" ixz="0.0" iyy=".0010" iyz="0.0" izz=".0010"/>
-    </inertial>
-    <visual>
-      <geometry>
-        <mesh filename="package://r2_description/meshes/Finger_Dist.dae"/>
-      </geometry>
-      <origin xyz="0.0 0.0 0.0" rpy="0 -1.57 0"/>
-    </visual>
-    <collision>
-      <geometry>
-        <mesh filename="package://r2_description/meshes/Finger_Dist.dae" scale="0.9 0.9 0.9"/>
+      <mass value=".001"/>
+      <inertia ixx=".0010" ixy="0.0" ixz="0.0" iyy=".0010" iyz="0.0" izz=".0010"/>
+    </inertial>
+    <visual>
+      <geometry>
+        <mesh filename="package://r2_description/meshes/Finger_Dist.dae"/>
+      </geometry>
+      <origin xyz="0.0 0.0 0.0" rpy="0 -1.57 0"/>
+    </visual>
+    <collision>
+      <geometry>
+        <mesh filename="package://r2_description/meshes/Finger_Dist.dae"/>
       </geometry>
       <origin xyz="0.0 0.0 0.0" rpy="0 -1.57 0"/>
@@ -484,5 +484,5 @@
   <link name="${robot_name}right_ring_tip">
     <inertial>
-      <mass value=".05"/>
+      <mass value=".001"/>
       <inertia ixx=".0010" ixy="0.0" ixz="0.0" iyy=".0010" iyz="0.0" izz=".0010"/>
     </inertial>
@@ -490,16 +490,16 @@
   <link name="${robot_name}right_little_proximal">
     <inertial>
-      <mass value=".05"/>
-      <inertia ixx=".0010" ixy="0.0" ixz="0.0" iyy=".0010" iyz="0.0" izz=".0010"/>
-    </inertial>
-    <visual>
-      <geometry>
-        <mesh filename="package://r2_description/meshes/Finger_Proximal.dae"/>
-      </geometry>
-      <origin xyz="0.0 0.0 0.0" rpy="0 0 1.57"/>
-    </visual>
-    <collision>
-      <geometry>
-        <mesh filename="package://r2_description/meshes/Finger_Proximal.dae" scale="0.9 0.9 0.9"/>
+      <mass value=".001"/>
+      <inertia ixx=".0010" ixy="0.0" ixz="0.0" iyy=".0010" iyz="0.0" izz=".0010"/>
+    </inertial>
+    <visual>
+      <geometry>
+        <mesh filename="package://r2_description/meshes/Finger_Proximal.dae"/>
+      </geometry>
+      <origin xyz="0.0 0.0 0.0" rpy="0 0 1.57"/>
+    </visual>
+    <collision>
+      <geometry>
+        <mesh filename="package://r2_description/meshes/Finger_Proximal.dae"/>
       </geometry>
       <origin xyz="0.0 0.0 0.0" rpy="0 0 1.57"/>
@@ -516,16 +516,16 @@
   <link name="${robot_name}right_little_medial">
     <inertial>
-      <mass value=".05"/>
-      <inertia ixx=".0010" ixy="0.0" ixz="0.0" iyy=".0010" iyz="0.0" izz=".0010"/>
-    </inertial>
-    <visual>
-      <geometry>
-        <mesh filename="package://r2_description/meshes/Finger_Mid.dae"/>
-      </geometry>
-      <origin xyz="0.0 0.0 0.0" rpy="3.14 0 1.57"/>
-    </visual>
-    <collision>
-      <geometry>
-        <mesh filename="package://r2_description/meshes/Finger_Mid.dae" scale="0.9 0.9 0.9"/>
+      <mass value=".001"/>
+      <inertia ixx=".0010" ixy="0.0" ixz="0.0" iyy=".0010" iyz="0.0" izz=".0010"/>
+    </inertial>
+    <visual>
+      <geometry>
+        <mesh filename="package://r2_description/meshes/Finger_Mid.dae"/>
+      </geometry>
+      <origin xyz="0.0 0.0 0.0" rpy="3.14 0 1.57"/>
+    </visual>
+    <collision>
+      <geometry>
+        <mesh filename="package://r2_description/meshes/Finger_Mid.dae"/>
       </geometry>
       <origin xyz="0.0 0.0 0.0" rpy="3.14 0 1.57"/>
@@ -542,16 +542,16 @@
   <link name="${robot_name}right_little_distal">
     <inertial>
-      <mass value=".05"/>
-      <inertia ixx=".0010" ixy="0.0" ixz="0.0" iyy=".0010" iyz="0.0" izz=".0010"/>
-    </inertial>
-    <visual>
-      <geometry>
-        <mesh filename="package://r2_description/meshes/Finger_Dist.dae"/>
-      </geometry>
-      <origin xyz="0.0 0.0 0.0" rpy="0 -1.57 0"/>
-    </visual>
-    <collision>
-      <geometry>
-        <mesh filename="package://r2_description/meshes/Finger_Dist.dae" scale="0.9 0.9 0.9"/>
+      <mass value=".001"/>
+      <inertia ixx=".0010" ixy="0.0" ixz="0.0" iyy=".0010" iyz="0.0" izz=".0010"/>
+    </inertial>
+    <visual>
+      <geometry>
+        <mesh filename="package://r2_description/meshes/Finger_Dist.dae"/>
+      </geometry>
+      <origin xyz="0.0 0.0 0.0" rpy="0 -1.57 0"/>
+    </visual>
+    <collision>
+      <geometry>
+        <mesh filename="package://r2_description/meshes/Finger_Dist.dae"/>
       </geometry>
       <origin xyz="0.0 0.0 0.0" rpy="0 -1.57 0"/>
@@ -565,5 +565,5 @@
   <link name="${robot_name}right_little_tip">
     <inertial>
-      <mass value=".05"/>
+      <mass value=".001"/>
       <inertia ixx=".0010" ixy="0.0" ixz="0.0" iyy=".0010" iyz="0.0" izz=".0010"/>
     </inertial>

Commit message: Slow down arms

File: r2_description/urdf/r2.left_arm.xacro (robot description, xacro)
@@ -21,5 +21,5 @@
     <axis xyz="0 0 1"/>
     <dynamics damping="${left_arm_j0_damping}" friction="${left_arm_j0_friction}"/>
-    <limit effort="100.0" lower="-1.57" upper="1.57" velocity="10"/>
+    <limit effort="100.0" lower="-1.57" upper="1.57" velocity="1"/>
   </joint>
   <link name="${robot_name}left_shoulder_roll">
@@ -49,5 +49,5 @@
     <axis xyz="0 0 1"/>
     <dynamics damping="${left_arm_j1_damping}" friction="${left_arm_j1_friction}"/>
-    <limit effort="100.0" lower="-1.66" upper=".175" velocity="10"/>
+    <limit effort="100.0" lower="-1.66" upper=".175" velocity="1"/>
   </joint>
   <link name="${robot_name}left_shoulder_pitch">
@@ -77,5 +77,5 @@
     <axis xyz="0 0 1"/>
     <dynamics damping="${left_arm_j2_damping}" friction="${left_arm_j2_friction}"/>
-    <limit effort="100.0" lower="-4.89" upper="-0.79" velocity="10"/>
+    <limit effort="100.0" lower="-4.89" upper="-0.79" velocity="1"/>
   </joint>
   <link name="${robot_name}left_upper_arm">
@@ -105,5 +105,5 @@
     <axis xyz="0 0 1"/>
     <dynamics damping="${left_arm_j3_damping}" friction="${left_arm_j3_friction}"/>
-    <limit effort="100.0" lower="-2.79" upper="-.087" velocity="10"/>
+    <limit effort="100.0" lower="-2.79" upper="-.087" velocity="1"/>
   </joint>
   <link name="${robot_name}left_elbow">
@@ -133,5 +133,5 @@
     <axis xyz="0 0 1"/>
     <dynamics damping="${left_arm_j4_damping}" friction="${left_arm_j4_friction}"/>
-    <limit effort="100.0" lower="-1.3" upper="4.45" velocity="10"/>
+    <limit effort="100.0" lower="-1.3" upper="4.45" velocity="1"/>
   </joint>
   <link name="${robot_name}left_lower_arm">
@@ -161,5 +161,5 @@
     <axis xyz="0 0 1"/>
     <dynamics damping="${left_arm_j5_damping}" friction="${left_arm_j5_friction}"/>
-    <limit effort="100.0" lower="-1.22" upper="1.22" velocity="10"/>
+    <limit effort="100.0" lower="-1.22" upper="1.22" velocity="1"/>
   </joint>
   <link name="${robot_name}left_wrist_pitch">
@@ -176,5 +176,5 @@
     <axis xyz="0 0 1"/>
     <dynamics damping="${left_arm_j6_damping}" friction="${left_arm_j6_friction}"/>
-    <limit effort="100.0" lower="-0.785" upper="0.785" velocity="10"/>
+    <limit effort="100.0" lower="-0.785" upper="0.785" velocity="1"/>
   </joint>
   <link name="${robot_name}left_wrist_yaw">

File: r2_description/urdf/r2.right_arm.xacro (robot description, xacro)
@@ -21,5 +21,5 @@
     <axis xyz="0 0 1"/>
     <dynamics damping="${right_arm_j0_damping}" friction="${right_arm_j0_friction}"/>
-    <limit effort="100.0" lower="-1.57" upper="1.57" velocity="10"/>
+    <limit effort="100.0" lower="-1.57" upper="1.57" velocity="1"/>
   </joint>
   <link name="${robot_name}right_shoulder_roll">
@@ -49,5 +49,5 @@
     <axis xyz="0 0 1"/>
     <dynamics damping="${right_arm_j1_damping}" friction="${right_arm_j1_friction}"/>
-    <limit effort="100.0" lower="-1.66" upper=".175" velocity="10"/>
+    <limit effort="100.0" lower="-1.66" upper=".175" velocity="1"/>
   </joint>
   <link name="${robot_name}right_shoulder_pitch">
@@ -77,5 +77,5 @@
     <axis xyz="0 0 1"/>
     <dynamics damping="${right_arm_j2_damping}" friction="${right_arm_j2_friction}"/>
-    <limit effort="100.0" lower="0.785" upper="4.89" velocity="10"/>
+    <limit effort="100.0" lower="0.785" upper="4.89" velocity="1"/>
   </joint>
   <link name="${robot_name}right_upper_arm">
@@ -105,5 +105,5 @@
     <axis xyz="0 0 1"/>
     <dynamics damping="${right_arm_j3_damping}" friction="${right_arm_j3_friction}"/>
-    <limit effort="100.0" lower="-2.79" upper="-.087" velocity="10"/>
+    <limit effort="100.0" lower="-2.79" upper="-.087" velocity="1"/>
   </joint>
   <link name="${robot_name}right_elbow">
@@ -133,5 +133,5 @@
     <axis xyz="0 0 1"/>
     <dynamics damping="${right_arm_j4_damping}" friction="${right_arm_j4_friction}"/>
-    <limit effort="100.0" lower="-4.45" upper="1.31" velocity="10"/>
+    <limit effort="100.0" lower="-4.45" upper="1.31" velocity="1"/>
   </joint>
   <link name="${robot_name}right_lower_arm">
@@ -161,5 +161,5 @@
     <axis xyz="0 0 1"/>
     <dynamics damping="${right_arm_j5_damping}" friction="${right_arm_j5_friction}"/>
-    <limit effort="100.0" lower="-1.22" upper="1.22" velocity="10"/>
+    <limit effort="100.0" lower="-1.22" upper="1.22" velocity="1"/>
   </joint>
   <link name="${robot_name}right_wrist_pitch">
@@ -176,5 +176,5 @@
     <axis xyz="0 0 1"/>
     <dynamics damping="${right_arm_j6_damping}" friction="${right_arm_j6_friction}"/>
-    <limit effort="100.0" lower="-0.785" upper="0.785" velocity="10"/>
+    <limit effort="100.0" lower="-0.785" upper="0.785" velocity="1"/>
   </joint>
   <link name="${robot_name}right_wrist_yaw">

Commit message: Fixed collision models on arm

File: r2_description/urdf/r2.left_arm.xacro (robot description, xacro)
@@ -33,5 +33,5 @@
     <!-- <collision>
       <geometry>
-        <mesh filename="package://r2_description/meshes/Left_Shoulder_Upper.dae" scale="0.7 0.7 0.7"/>
+        <mesh filename="package://r2_description/meshes/Left_Shoulder_Upper.dae" />
       </geometry>
       <origin rpy="0 0 1.57" xyz="0 0 .08"/>
@@ -89,5 +89,5 @@
     <collision>
       <geometry>
-        <mesh filename="package://r2_description/meshes/Left_Upper_Arm.dae" scale="0.8 0.8 0.8"/>
+        <mesh filename="package://r2_description/meshes/Left_Upper_Arm.dae" />
       </geometry>
       <origin rpy="0 0 3.14" xyz="0 0 .1016"/>

Commit message: Add shoulder collision models back in

File: r2_description/urdf/r2.left_arm.xacro (robot description, xacro)
@@ -31,10 +31,10 @@
       <origin rpy="0 0 1.57" xyz="0 0 .08"/>
     </visual>
-    <!-- <collision>
+    <collision>
       <geometry>
         <mesh filename="package://r2_description/meshes/Left_Shoulder_Upper.dae" />
       </geometry>
       <origin rpy="0 0 1.57" xyz="0 0 .08"/>
-    </collision> -->
+    </collision>
     <inertial>
 	<origin xyz="-0.0089916 -0.00131572   0.10287   "/>
@@ -59,10 +59,10 @@
       <origin rpy=".0 0 -1.57" xyz="0 0 0"/>
     </visual>
-    <!-- <collision>
+    <collision>
       <geometry>
         <mesh filename="package://r2_description/meshes/Left_Shoulder_Lower.dae"/>
       </geometry>
       <origin rpy=".0 0 -1.57" xyz="0 0 0"/>
-    </collision> -->
+    </collision>
      <inertial>
         <origin xyz="0.037084 -0.00028448   0.0077978   "/>

File: r2_description/urdf/r2.right_arm.xacro (robot description, xacro)
@@ -31,10 +31,10 @@
       <origin rpy="0 0 2.25" xyz="0 0 .0254"/>
     </visual>
-    <!-- <collision>
+    <collision>
       <geometry>
         <mesh filename="package://r2_description/meshes/Right_Shoulder_Upper.dae"/>
       </geometry>
       <origin rpy="0 0 2.35" xyz="0 0 .0254"/>
-    </collision> -->
+    </collision>
     <inertial>
         <origin xyz="0.0089916 -0.00131572  0.10287"/>
@@ -59,10 +59,10 @@
       <origin rpy=".0 0 1.57" xyz="0 0 0"/>
     </visual>
-  <!--   <collision>
+    <collision>
       <geometry>
         <mesh filename="package://r2_description/meshes/Right_Shoulder_Lower.dae"/>
       </geometry>
       <origin rpy=".0 0 1.57" xyz="0 0 0"/>
-    </collision> -->
+    </collision>
      <inertial>
         <origin xyz="0.0077978 0.037084 0.00028448"/>
