Commit message: Right shoulder collision and vidsual had different origins for same mesh

File: r2_description/urdf/r2.right_arm.xacro (robot description, xacro)
@@ -35,5 +35,5 @@
         <mesh filename="package://r2_description/meshes/Right_Shoulder_Upper.dae"/>
       </geometry>
-      <origin rpy="0 0 2.35" xyz="0 0 .0254"/>
+      <origin rpy="0 0 2.25" xyz="0 0 .0254"/>
     </collision>
     <inertial>
